File: power/48-12.kicad_sch (KiCad schematic)
At the start: 13 parts, among them U1 BMR4800116/005, U2 HO150-NP

Commit message: work
Parts:
- R5: now not fitted
- U1: value BMR4800116/005 -> MPQ1500-12V125-L48NBMC
Connections:
- net 5V_PRESENSE is gone; now on net +5V: R10.1
- net 12V_CURRENT_VREF renamed +1V25
Other:
- note added: "PIN COMPATIBLE BRICKS (48-12V): BMR4800116/005 (1300W) MPQ1500-12V125-L48NBMC (1500W)"
- note removed: "1.3V Ideal"
- moved on the sheet: C12, C13, C14, C15, C16, C17, C18, C19, R10, R4, U2

Commit message: update
Parts:
- removed R10: 22k, Resistor_SMD:R_0603_1608Metric, symbol Device:R_Small
- added J9: BMR_I2C, Connector_PinHeader_2.54mm:PinHeader_1x03_P2.54mm_Vertical, symbol Connector:Conn_01x03_Pin
- added R1: 10k, Resistor_SMD:R_0603_1608Metric, symbol Device:R_Small
- added TP_12V_CURRENT_VOUT1, TP_12V_OCD1, TP_12V_PG1: TestPoint, TestPoint:TestPoint_THTPad_2.5x2.5mm_Drill1.2mm, symbol Connector:TestPoint
- U2: footprint custom:LEM_HO150-NP -> power_symbols:LEM_HO150-NP
- renumbered C12 to C11, C13 to C12, C14 to C13, C15 to C14, C16 to C15, C17 to C16, C18 to C17, C19 to C18, R4 to R2, R5 to R3
Connections:
- net +5V: now also R1.1
- net 12V_CURRENT_OCD: now also R1.2, TP_12V_OCD1.1
- net 12V_CURRENT_VOUT: now also TP_12V_CURRENT_VOUT1.1
- net 12V_GND: now also J9.3 (Pin_3)
- net BMR_SCL: now also J9.2 (Pin_2)
- net BMR_SDA: now also J9.1 (Pin_1)
- net ~{BMR_PG}: now also TP_12V_PG1.1
Other:
- note added: "PIN COMPATIBLE BRICKS (48-12V): BMR4800116/005 (1300W) MPQ1500-12V125-L48NBMC (1500W) Pins 9, 10, 15 are not fitted on MPQ1500"
- note removed: "PIN COMPATIBLE BRICKS (48-12V): BMR4800116/005 (1300W) MPQ1500-12V125-L48NBMC (1500W)"
- moved on the sheet: C11, C12, C13, C14, C15, C16, C17, C18, R2, R3, U1, U2

Commit message: final
Parts:
- C11, C12: value C_Polarized_Small -> 2.2mF 16V poly; footprint Capacitor_THT:CP_Radial_D10.0mm_P5.00mm -> Capacitor_THT:CP_Radial_D18.0mm_P7.50mm; LCSC (none) -> C240374; MPN (none) -> GR1J222MM300A00CV0
- C13, C14, C15, C16, C17, C18: value C_Small -> 10uF; LCSC (none) -> C96446; MPN (none) -> CL10A106MA8NRNC
- J7: renamed from J9; MPN (none) -> -
- R1, R2, R3: LCSC (none) -> C25804; MPN (none) -> 0603WAF1002T5E
- TP_12V_CURRENT_VOUT1, TP_12V_OCD1, TP_12V_PG1: MPN (none) -> -
- U1: MPN (none) -> MPQ1500-12V125-L48NBMC
- U2: MPN (none) -> HO 150-NP-0100
