File: power/STM.kicad_sch (KiCad schematic)
At the start: 15 parts, among them J6 SWD, SW1 SW_Push, U7 STM32G431KBTx, U8 AZ1117-3.3

Commit message: work
Parts:
- added C23, C25: 100nF, Capacitor_SMD:C_0603_1608Metric, symbol Device:C_Small
- added D1: 48V (BLUE), symbol Device:LED
- added D2: 5V (GREEN), symbol Device:LED
- added D3: 12V (RED), symbol Device:LED
- added D4: 5V_PG (GREEN), symbol Device:LED
- added D5: 12V_PG (RED), symbol Device:LED
- added D6: 3V3 (PURPLE), symbol Device:LED
- added R1, R16: 1k2 1W, symbol Device:R_Small
- added R17, R2, R20, R3: 120R, symbol Device:R_Small
- added R18: 500R, symbol Device:R_Small
Connections:
- net 5V_CURRENT_VREF is gone; now on net +1V25: U7.12 (PA7)
- net +3V3: now also C25.1, D6.2 (A)
- net +5V: now also C23.1, D2.2 (A), D5.2 (A)
- net 12V_GND: now also C23.2, C25.2, R17.2, R18.2, R20.2, R3.2
- net ~{BMR_PG}: now also R2.2
- net 12V_CURRENT_VREF renamed +1V25
- net RPM_PG renamed 5V_PG
- net 5V_PG: now also D4.2 (A)
- new net: D3.1 (K), R18.1
- new net: D6.1 (K), R20.1
- new net: D4.1 (K), R3.1
- new net: R1.1, R16.2
- new net: D5.1 (K), R2.1
- new net: D2.1 (K), R17.1
- new net: D1.1 (K), R16.1
- new net +12V: D3.2 (A)
- new net +48V: D1.2 (A)
- new net 48V_GND: R1.2
Other:
- moved on the sheet: C20, C21, C22, C35, C36, C37, J6, R11, R12, R13, R14, R15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

Commit message: update
Parts:
- removed C21, C22: 10uF, Capacitor_SMD:C_0603_1608Metric, symbol Device:C_Small
- removed C23, C25: 100nF, Capacitor_SMD:C_0603_1608Metric, symbol Device:C_Small
- removed R1: 1k2 1W, symbol Device:R_Small
- removed R20: 120R, symbol Device:R_Small
- removed U8: AZ1117-3.3, Package_TO_SOT_SMD:SOT-223-3_TabPin2, symbol Regulator_Linear:AZ1117-3.3
- added C30, C31, C33, C34: 10uF, Capacitor_SMD:C_0603_1608Metric, symbol Device:C_Small
- added J7: I2C, Connector_PinHeader_2.54mm:PinHeader_1x03_P2.54mm_Vertical, symbol Connector:Conn_01x03_Pin
- added R10, R11: 10k, Resistor_SMD:R_0603_1608Metric, symbol Device:R_Small
- added R21, R22, R23: 680R 1/4W 0603, Resistor_SMD:R_0603_1608Metric, symbol Device:R_Small
- added TP_12V_VDETECT1, TP_1V1, TP_3V1, TP_5V_VDETECT1: TestPoint, TestPoint:TestPoint_THTPad_2.5x2.5mm_Drill1.2mm, symbol Connector:TestPoint
- added U5: TPS7A24125DBVR, Package_TO_SOT_SMD:SOT-23-5, symbol custom:TPS7A24125DBVR
- added U6: TPS7A2433DBVR, Package_TO_SOT_SMD:SOT-23-5, symbol custom:TPS7A2433DBVR
- C32: renamed from C20; footprint (none) -> Capacitor_SMD:C_0603_1608Metric
- D1, D5: footprint (none) -> LED_SMD:LED_0603_1608Metric
- D2: renamed from D3; footprint (none) -> LED_SMD:LED_0603_1608Metric
- D3: renamed from D2; footprint (none) -> LED_SMD:LED_0603_1608Metric
- D4: renamed from D6; footprint (none) -> LED_SMD:LED_0603_1608Metric
- D6: renamed from D4; footprint (none) -> LED_SMD:LED_0603_1608Metric
- J8: renamed from J6; footprint (none) -> Connector_PinHeader_2.54mm:PinHeader_1x05_P2.54mm_Vertical
- R16: value 1k2 1W -> 680R 1/4W 0603; footprint (none) -> Resistor_SMD:R_0603_1608Metric
- R17: renamed from R18; footprint (none) -> Resistor_SMD:R_0603_1608Metric
- R18: renamed from R17; footprint (none) -> Resistor_SMD:R_0603_1608Metric
- R19: renamed from R2; footprint (none) -> Resistor_SMD:R_0603_1608Metric
- R20: renamed from R3; footprint (none) -> Resistor_SMD:R_0603_1608Metric
- R9: renamed from R15; footprint (none) -> Resistor_SMD:R_0603_1608Metric
- SW1: footprint (none) -> power_symbols:TS04-66-70-BK-160-SMT
- renumbered C35 to C27, C36 to C28, C37 to C29, R11 to R12, R12 to R13, R13 to R14, R14 to R15
Connections:
- net +1V25: now also C30.1, TP_1V1.1, U5.5 (V_{OUT})
- net +3V3: now also C33.1, R10.1, R11.1, TP_3V1.1, U6.5 (V_{OUT})
- net +5V: now also C31.1, C34.1, U5.1 (V_{IN}), U5.3 (EN), U6.1 (V_{IN}), U6.3 (EN)
- net 12V_GND: now also D4.1 (K), C30.2, C31.2, C33.2, C34.2, J7.3 (Pin_3), U5.2 (GND), U6.2 (GND)
- net 12V_VDETECT: now also TP_12V_VDETECT1.1
- net 48V_GND: now also R23.2
- net 5V_VDETECT: now also TP_5V_VDETECT1.1
- net I2C_SCL: now also J7.2 (Pin_2), R11.2
- net I2C_SDA: now also J7.1 (Pin_1), R10.2
- net at R16.2: now also R21.1
- new net: R22.2, R23.1
- new net: R21.2, R22.1
Other:
- note added: "TS04-66-70-BK-160-SMT"
- moved on the sheet: J8, R12, R13, R14, R15

Commit message: final
Parts:
- added R12, R13: 0R, Resistor_SMD:R_0603_1608Metric, symbol Device:R_Small
- C27: value C_Small -> 0.1uF; LCSC (none) -> C14663; MPN (none) -> CC0603KRX7R9BB104
- C28, C29: value C_Small -> 1uF; LCSC (none) -> C15849; MPN (none) -> CL10A105KB8NNNC
- C30, C31, C33, C34: LCSC (none) -> C96446; MPN (none) -> CL10A106MA8NRNC
- C32: LCSC (none) -> C5360803; MPN (none) -> TCC0603X5R335M250CT
- D1: value 48V (BLUE) -> BLUE; LCSC (none) -> C965807; MPN (none) -> XL-1608UBC-04
- D2: value 12V (RED) -> RED; LCSC (none) -> C965799; MPN (none) -> XL-1608SURC-06
- D3: value 5V (GREEN) -> GREEN; LCSC (none) -> C965804; MPN (none) -> XL-1608UGC-04
- D4: value 3V3 (PURPLE) -> PURPLE; LCSC (none) -> C7371898; MPN (none) -> XL-1608UVC-04
- D5: value 12V_PG (RED) -> RED; LCSC (none) -> C965799; MPN (none) -> XL-1608SURC-06
- D6: value 5V_PG (GREEN) -> GREEN; LCSC (none) -> C965804; MPN (none) -> XL-1608UGC-04
- J8: renamed from J7; MPN (none) -> -
- J9: renamed from J8; MPN (none) -> -
- R10, R11, R9: LCSC (none) -> C25804; MPN (none) -> 0603WAF1002T5E
- R14: renamed from R12; LCSC (none) -> C22984; MPN (none) -> 0603WAF3002T5E
- R15: renamed from R13; LCSC (none) -> C25804; MPN (none) -> 0603WAF1002T5E
- R16: renamed from R14; LCSC (none) -> C25804; MPN (none) -> 0603WAF1002T5E
- R17: renamed from R15; LCSC (none) -> C22809; MPN (none) -> 0603WAF1502T5E
- R18: renamed from R16; value 680R 1/4W 0603 -> 680R 1/4W; LCSC (none) -> C445820; MPN (none) -> ERJPA3J681V
- R19: renamed from R17; value 500R -> 680R 1/4W; LCSC (none) -> C445820; MPN (none) -> ERJPA3J681V
- R20: renamed from R18; LCSC (none) -> C22787; MPN (none) -> 0603WAF1200T5E
- R21: renamed from R19; LCSC (none) -> C22787; MPN (none) -> 0603WAF1200T5E
- R22: renamed from R20; LCSC (none) -> C22787; MPN (none) -> 0603WAF1200T5E
- R23: renamed from R21; value 680R 1/4W 0603 -> 680R 1/4W; LCSC (none) -> C445820; MPN (none) -> ERJPA3J681V
- R24: renamed from R22; value 680R 1/4W 0603 -> 680R 1/4W; LCSC (none) -> C445820; MPN (none) -> ERJPA3J681V
- R25: renamed from R23; value 680R 1/4W 0603 -> 680R 1/4W; LCSC (none) -> C445820; MPN (none) -> ERJPA3J681V
- SW1: LCSC (none) -> C455109; MPN (none) -> TS04-66-70-BK-160-SMT
- TP_12V_VDETECT1, TP_5V_VDETECT1: MPN (none) -> -
- TP_1V25_1: renamed from TP_1V1; MPN (none) -> -
- TP_3V_1: renamed from TP_3V1; MPN (none) -> -
- U5: MPN (none) -> TPS7A24125DBVR
- U6: MPN (none) -> TPS7A2433DBVR
- U7: MPN (none) -> STM32G431KBT6
Connections:
- net I2C_SCL: now also R13.1; no longer U7.19 (PA9)
- net I2C_SDA: now also R12.2; no longer U7.18 (PA8)
- new net: R12.1, U7.18 (PA8)
- new net: R13.2, U7.19 (PA9)
