File: power/power.kicad_pcb (KiCad board)
At the start: 2 copper layers, 108.2 x 81.5 mm, 2 parts, among them J1 ET60T-D04-3-08-D04-X-R1-S, J2 796636-6

Commit message: work
Parts:
- added C1: C_Polarized_Small, Capacitor_THT:CP_Radial_D18.0mm_P7.50mm, F.Cu at (47.5, 102.5)
- added C10: C_Small, Capacitor_SMD:C_0603_1608Metric, F.Cu at (43.2, 147.5)
- added C11: C_Small, Capacitor_SMD:C_0603_1608Metric, F.Cu at (43.2, 145.0)
- added C12: C_Polarized_Small, Capacitor_THT:CP_Radial_D18.0mm_P7.50mm, F.Cu at (92.5, 132.0)
- added C13: C_Polarized_Small, Capacitor_THT:CP_Radial_D18.0mm_P7.50mm, F.Cu at (92.5, 112.5)
- added C14: C_Polarized_Small, Capacitor_THT:CP_Radial_D10.0mm_P5.00mm, F.Cu at (72.9, 136.0)
- added C15: C_Polarized_Small, Capacitor_THT:CP_Radial_D10.0mm_P5.00mm, F.Cu at (72.9, 124.5)
- added C16: C_Polarized_Small, Capacitor_THT:CP_Radial_D10.0mm_P5.00mm, F.Cu at (72.9, 112.9)
- added C17: C_Polarized_Small, Capacitor_THT:CP_Radial_D10.0mm_P5.00mm, F.Cu at (72.9, 101.3)
- added C18: C_Polarized_Small, Capacitor_THT:CP_Radial_D10.0mm_P5.00mm, F.Cu at (72.9, 89.8)
- added C19: C_Polarized_Small, Capacitor_THT:CP_Radial_D10.0mm_P5.00mm, F.Cu at (72.7, 78.5)
- added C2: C_Polarized_Small, Capacitor_THT:CP_Radial_D18.0mm_P7.50mm, F.Cu at (47.5, 83.0)
- added C20: C_Small, Capacitor_SMD:C_0603_1608Metric, F.Cu at (88.4, 101.3)
- added C21: C_Small, Capacitor_SMD:C_0603_1608Metric, F.Cu at (88.4, 98.8)
- added C22: C_Small, Capacitor_SMD:C_0603_1608Metric, F.Cu at (88.4, 96.3)
- added C23: C_Small, Capacitor_SMD:C_0603_1608Metric, F.Cu at (88.4, 93.8)
- added C24: C_Small, Capacitor_SMD:C_0603_1608Metric, F.Cu at (88.4, 91.2)
- added C25: C_Small, Capacitor_SMD:C_0603_1608Metric, F.Cu at (88.4, 88.7)
- added C26: C_Small, Capacitor_SMD:C_0603_1608Metric, F.Cu at (88.4, 86.2)
- added C27: C_Small, Capacitor_SMD:C_0603_1608Metric, F.Cu at (88.4, 83.7)
- added C28: C_Small, Capacitor_SMD:C_0603_1608Metric, F.Cu at (88.4, 81.2)
- added C29: C_Small, Capacitor_SMD:C_0603_1608Metric, F.Cu at (88.4, 78.7)
- added C3: C_Polarized_Small, Capacitor_THT:CP_Radial_D8.0mm_P5.00mm, F.Cu at (45.9, 137.6)
- added C30: C_Polarized_Small, Capacitor_THT:CP_Radial_D10.0mm_P5.00mm, F.Cu at (115.1, 106.5)
- added C31: C_Polarized_Small, Capacitor_THT:CP_Radial_D10.0mm_P5.00mm, F.Cu at (115.1, 118.0)
- added C32: C_Polarized_Small, Capacitor_THT:CP_Radial_D10.0mm_P5.00mm, F.Cu at (115.1, 129.6)
- added C33: C_Polarized_Small, Capacitor_THT:CP_Radial_D10.0mm_P5.00mm, F.Cu at (115.1, 141.2)
- added C34: C_Small, Capacitor_SMD:C_0603_1608Metric, F.Cu at (117.8, 148.5)
- added C35: C_Small, Capacitor_SMD:C_0603_1608Metric, F.Cu at (117.8, 151.0)
- added C36: C_Small, Capacitor_SMD:C_0603_1608Metric, F.Cu at (117.8, 153.5)
- added C37: C_Small, Capacitor_SMD:C_0603_1608Metric, F.Cu at (117.8, 156.0)
- added C38: C_Small, Capacitor_SMD:C_0603_1608Metric, F.Cu at (117.8, 158.5)
- added C39: C_Small, Capacitor_SMD:C_0603_1608Metric, F.Cu at (117.8, 161.0)
- added C4: C_Polarized_Small, Capacitor_THT:CP_Radial_D8.0mm_P5.00mm, F.Cu at (45.9, 128.1)
- added C40: C_Small, Capacitor_SMD:C_0603_1608Metric, F.Cu at (117.8, 163.5)
- added C5: C_Polarized_Small, Capacitor_THT:CP_Radial_D8.0mm_P5.00mm, F.Cu at (45.9, 118.5)
- added C6: C_Small, Capacitor_SMD:C_0603_1608Metric, F.Cu at (43.2, 157.6)
- added C7: C_Small, Capacitor_SMD:C_0603_1608Metric, F.Cu at (43.2, 155.0)
- added C8: C_Small, Capacitor_SMD:C_0603_1608Metric, F.Cu at (43.2, 152.5)
- added C9: C_Small, Capacitor_SMD:C_0603_1608Metric, F.Cu at (43.2, 150.0)
- added G1: LOGO, custom:logo, F.Cu at (104.0, 103.5)
- added R1: 10k, Resistor_SMD:R_0603_1608Metric, F.Cu at (112.0, 156.7)
- added U1: BMR4912510/871, power_symbols:BMR491_FPM, F.Cu at (55.6, 155.6)
- added U2: RPM5.0-6.0, power_symbols:RPM5.0-6.0, F.Cu at (110.5, 92.0)
- moved J2 61.0 mm to (56.2, 66.5), turned to 180 degrees
- moved J1 7.49 mm to (160.6, 106.1), turned to 90 degrees
Connections:
- J1 pad 04: unconnected-(J1-Pad04) -> /RPM_PG
- J1 pad 05: unconnected-(J1-Pad05) -> /BMR_PG
- J1 pad 06: unconnected-(J1-Pad06) -> /BMR_SDA
- J1 pad 07: unconnected-(J1-Pad07) -> /BMR_SCL
- J1 pad 08: unconnected-(J1-Pad08) -> /BMR_SALERT
- J1 pad 09: 5V_GND -> 12V_GND
- J1 pad 10: 5V_GND -> 12V_GND
- J1 pad 17: 5V_GND -> 12V_GND
- J1 pad 18: 5V_GND -> 12V_GND
Routing:
- net 48V_GND: track 0.00 -> 233.3 mm, vias 0 -> 2
- net +48V: track 0.00 -> 222.0 mm, vias 0 -> 2
- net /BMR_SCL: track 0.00 -> 143.6 mm, vias 0 -> 2
- net /BMR_SALERT: track 0.00 -> 143.1 mm, vias 0 -> 1
- net /BMR_SDA: track 0.00 -> 135.9 mm, vias 0 -> 1
- net /BMR_PG: track 0.00 -> 128.4 mm, vias 0 -> 1
- net /RPM_PG: track 0.00 -> 78.9 mm, vias 0 -> 1
- net 12V_GND: track 0.00 -> 14.2 mm, vias 0 -> 232
- net Net-(U1-SA1): track 0.00 -> 4.66 mm
- net +12V: track 0.00 -> 3.80 mm
- added copper zone on F.Cu, net +48V
- added copper zone on F.Cu, net +5V
- added copper zone on F.Cu, net 12V_GND
- added copper zone on F.Cu, net 48V_GND
Other:
- board size 108.2 x 81.5 mm -> 143.2 x 125.1 mm

Commit message: stuff
Parts:
- removed C12, C13: C_Polarized_Small, Capacitor_THT:CP_Radial_D18.0mm_P7.50mm
- removed C16, C17, C18, C19: C_Polarized_Small, Capacitor_THT:CP_Radial_D10.0mm_P5.00mm
- removed U1: BMR4912510/871, power_symbols:BMR491_FPM
- added H1: MountingHole, MountingHole:MountingHole_3.2mm_M3, F.Cu at (30.2, 142.2)
- added H2: MountingHole, MountingHole:MountingHole_3.2mm_M3, F.Cu at (67.2, 27.8)
- added H3: MountingHole, MountingHole:MountingHole_3.2mm_M3, F.Cu at (147.0, 142.0)
- added R2: 10k, Resistor_SMD:R_0603_1608Metric, F.Cu at (111.9, 125.3)
- added U3: BMR4800116/005, power_symbols:BMR491_FPM, F.Cu at (55.0, 118.0)
- moved C38 92.0 mm to (120.4, 66.5)
- moved C34 92.0 mm to (120.4, 56.5)
- moved C35 92.0 mm to (120.4, 59.0)
- moved C36 92.0 mm to (120.4, 61.5)
- moved C39 92.0 mm to (120.4, 69.1)
- moved C40 92.0 mm to (120.4, 71.6)
- moved C37 92.0 mm to (120.4, 64.0)
- moved C14 54.9 mm to (89.0, 83.5)
- moved G1 43.0 mm to (144.5, 118.0)
- moved C30 41.7 mm to (115.2, 64.8), turned to 180 degrees
- moved C31 41.5 mm to (115.2, 76.5), turned to 180 degrees
- moved C32 41.5 mm to (115.2, 88.1), turned to 180 degrees
- moved C33 41.5 mm to (115.2, 99.7), turned to 180 degrees
- moved U2 39.8 mm to (109.9, 52.2)
- moved J1 39.2 mm to (144.9, 70.2)
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Connections:
- J1 pad 05: /BMR_PG -> /~{BMR_PG}
- J1 pad 08: /BMR_SALERT -> /~{BMR_SALERT}
Routing:
- net /BMR_SALERT: track 143.1 -> 0.00 mm, vias 1 -> 0
- net /BMR_PG: track 128.4 -> 0.00 mm, vias 1 -> 0
- net /~{BMR_SALERT}: track 0.00 -> 126.8 mm, vias 0 -> 1
- net /~{BMR_PG}: track 0.00 -> 121.3 mm, vias 0 -> 1
- net 48V_GND: track 233.3 -> 189.0 mm, vias 2 -> 9
- net +48V: track 222.0 -> 193.1 mm, vias 2 -> 0
- net /RPM_PG: track 78.9 -> 60.2 mm
- net /BMR_SCL: track 143.6 -> 127.1 mm
- net /BMR_SDA: track 135.9 -> 119.9 mm
- net Net-(U3-SA1): track 0.00 -> 6.06 mm
- net Net-(U3-SA0): track 4.66 -> 9.81 mm
- net +12V: track 3.80 -> 0.00 mm
- net 12V_GND: track 14.2 -> 10.5 mm, vias 232 -> 143
- net +5V: vias 0 -> 30
- added copper zone on B.Cu, net +5V
Other:
- board size 143.2 x 125.1 mm -> 127.8 x 125.1 mm

Commit message: update
Parts:
- removed C20, C21, C22, C23, C25, C27, C34, C38, C39, C40: C_Small, Capacitor_SMD:C_0603_1608Metric
- removed C30, C31: C_Polarized_Small, Capacitor_THT:CP_Radial_D10.0mm_P5.00mm
- added C12: C_Polarized_Small, Capacitor_THT:CP_Radial_D10.0mm_P5.00mm, F.Cu at (215.7, 44.7)
- added C13: C_Polarized_Small, Capacitor_THT:CP_Radial_D10.0mm_P5.00mm, F.Cu at (227.2, 44.7)
- added C16: C_Small, Capacitor_SMD:C_0603_1608Metric, F.Cu at (240.1, 42.3)
- added C17: C_Small, Capacitor_SMD:C_0603_1608Metric, F.Cu at (242.6, 42.3)
- added C18: C_Small, Capacitor_SMD:C_0603_1608Metric, F.Cu at (245.1, 42.3)
- added C19: C_Small, Capacitor_SMD:C_0603_1608Metric, F.Cu at (247.7, 42.3)
- added R10: 22k, Resistor_SMD:R_0603_1608Metric, F.Cu at (201.5, 75.5)
- added R11: 30k, Resistor_SMD:R_0603_1608Metric, F.Cu at (193.5, 97.6)
- added R12: 10k, Resistor_SMD:R_0603_1608Metric, F.Cu at (193.5, 100.1)
- added R13: 10k, Resistor_SMD:R_0603_1608Metric, F.Cu at (193.5, 102.6)
- added R14: 15k, Resistor_SMD:R_0603_1608Metric, F.Cu at (193.5, 105.1)
- added R3: 100k, Resistor_SMD:R_0603_1608Metric, F.Cu at (201.5, 73.2)
- added R4: 10k, Resistor_SMD:R_0603_1608Metric, F.Cu at (162.2, 29.0)
- added R5: 10k, Resistor_SMD:R_0603_1608Metric, F.Cu at (162.2, 31.5)
- added R6: 22k, Resistor_SMD:R_0603_1608Metric, F.Cu at (230.7, 91.8)
- added R7: 4k7, Resistor_SMD:R_0603_1608Metric, F.Cu at (233.9, 91.8)
- added R8: 100k, Resistor_SMD:R_0603_1608Metric, F.Cu at (237.2, 91.8)
- added R9: 22k, Resistor_SMD:R_0603_1608Metric, F.Cu at (231.8, 84.5)
- added U1: BMR4800116/005, power_symbols:BMR491_FPM, F.Cu at (157.3, 89.1)
- added U4: RPM5.0-6.0, power_symbols:RPM5.0-6.0, F.Cu at (224.0, 76.1)
- added U5: HO8-NP, Sensor_Current:LEM_HO8-NP, F.Cu at (243.3, 87.6)
- added U6: AZ431LANTR-G1, Package_TO_SOT_SMD:SOT-23-5, F.Cu at (230.5, 88.0)
- added U7: STM32G431KBTx, Package_QFP:LQFP-32_7x7mm_P0.8mm, F.Cu at (212.9, 90.7)
- added U8: AZ1117-3.3, Package_TO_SOT_SMD:SOT-223-3_TabPin2, F.Cu at (200.5, 104.4)
- C14, C15, C32, C33: value C_Polarized_Small -> C_Small; footprint Capacitor_THT:CP_Radial_D10.0mm_P5.00mm -> Capacitor_SMD:C_0603_1608Metric
- C24, C26: value C_Small -> C_Polarized_Small; footprint Capacitor_SMD:C_0603_1608Metric -> Capacitor_THT:CP_Radial_D10.0mm_P5.00mm
- R1: value 10k -> 22k
- R2: value 10k -> 4k7
- U2: value RPM5.0-6.0 -> HO150-NP; footprint power_symbols:RPM5.0-6.0 -> custom:LEM_HO150-NP
- U3: value BMR4800116/005 -> AZ431LANTR-G1; footprint power_symbols:BMR491_FPM -> Package_TO_SOT_SMD:SOT-23-5
- moved C24 162.0 mm to (245.8, 96.4), turned to -90 degrees
- moved C29 161.7 mm to (243.8, 91.5), turned to 90 degrees
- moved C28 158.7 mm to (241.2, 91.5), turned to 90 degrees
- moved C15 157.7 mm to (237.6, 42.3), turned to 90 degrees
- moved C26 152.6 mm to (235.0, 96.4), turned to -90 degrees
- moved C14 151.8 mm to (235.1, 42.3), turned to 90 degrees
- moved U3 151.5 mm to (201.6, 79.7)
- moved H1 135.3 mm to (121.0, 42.0), turned to 90 degrees
- moved C33 134.1 mm to (249.1, 91.5), turned to 90 degrees
- moved C32 131.3 mm to (246.6, 91.5), turned to 90 degrees
- moved C3 122.8 mm to (168.3, 97.8), turned to -90 degrees
- moved J1 114.5 mm to (259.5, 69.7)
- moved C4 113.3 mm to (158.8, 97.8), turned to -90 degrees
- moved R2 105.3 mm to (205.0, 76.0), turned to 0 degrees
- moved R1 105.0 mm to (205.0, 73.5), turned to 0 degrees
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Connections:
- C24 pad 1: +12V -> +5V
- C26 pad 1: +12V -> +5V
- C28 pad 1: +12V -> +5V
- C29 pad 1: +12V -> +5V
- C35 pad 1: +5V -> +3V3
- C36 pad 1: +5V -> +3V3
- C37 pad 1: +5V -> +3V3
- R1 pad 1: Net-(U3-SA0) -> /48-12/12V_CURRENT_VREF
- R1 pad 2: 12V_GND -> +5V
- R2 pad 1: Net-(U3-SA1) -> /48-12/12V_CURRENT_VREF
- R2 pad 2: 12V_GND -> Net-(U3-REF)
- U3 pad 1: +48V -> (no net)
- U3 pad 2: 48V_GND -> (no net)
- U3 pad 3: 48V_GND -> /48-12/12V_CURRENT_VREF
- U3 pad 4: 12V_GND -> Net-(U3-REF)
Routing:
- net /BMR_SCL: track 127.1 -> 0.00 mm, vias 2 -> 0
- net /~{BMR_SALERT}: track 126.8 -> 0.00 mm, vias 1 -> 0
- net /~{BMR_PG}: track 121.3 -> 0.00 mm, vias 1 -> 0
- net /BMR_SDA: track 119.9 -> 0.00 mm, vias 1 -> 0
- net 48V_GND: track 189.0 -> 124.8 mm, vias 9 -> 6
- net /RPM_PG: track 60.2 -> 0.00 mm, vias 1 -> 0
- net +48V: track 193.1 -> 135.1 mm
- net /12-5/5V_PRESENSE: track 0.00 -> 35.2 mm, vias 0 -> 1
- net /12-5/5V_CURRENT_VREF: track 0.00 -> 24.3 mm, vias 0 -> 1
- net Net-(U6-REF): track 0.00 -> 16.4 mm
- net 12V_GND: track 10.5 -> 25.7 mm, vias 143 -> 3
- net /12-5/5V_CURRENT_OCD: track 0.00 -> 10.0 mm
- net Net-(U3-SA0): track 9.81 -> 0.00 mm
- net /12-5/5V_CURRENT_VOUT: track 0.00 -> 9.11 mm
- net Net-(U3-SA1): track 6.06 -> 0.00 mm
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- added copper zone on F.Cu, net /12-5/5V_PRESENSE
- added copper zone on F.Cu, net /48-12/12V_PRESENSE
- added copper zone on B.Cu, net 48V_GND
- removed copper zone on B.Cu, net +5V
- removed copper zone on F.Cu, net 48V_GND
Other:
- board size 127.8 x 125.1 mm -> 165.1 x 98.5 mm

Commit message: work
Parts:
- added C21: 10uF, Capacitor_SMD:C_0603_1608Metric, F.Cu at (206.1, 74.9)
- added C22: 10uF, Capacitor_SMD:C_0603_1608Metric, F.Cu at (206.1, 77.4)
- added C23: 100nF, Capacitor_SMD:C_0603_1608Metric, F.Cu at (206.1, 79.9)
- added C25: 100nF, Capacitor_SMD:C_0603_1608Metric, F.Cu at (206.1, 82.4)
- added U3: TPS56A37RPAR, custom:TPS56A37RPAR, F.Cu at (213.1, 75.8)
Connections:
- J1 pad 04: /RPM_PG -> unconnected-(J1-Pad04)
- J1 pad 05: /~{BMR_PG} -> unconnected-(J1-Pad05)
- J1 pad 06: /BMR_SDA -> unconnected-(J1-Pad06)
- J1 pad 07: /BMR_SCL -> /STM_SDA
- J1 pad 08: /~{BMR_SALERT} -> /STM_SCL
- R11 pad 2: Net-(U7-PA4) -> /STM/12V_VDETECT
- R12 pad 1: Net-(U7-PA4) -> /STM/12V_VDETECT
- R13 pad 2: Net-(U7-PA3) -> /STM/5V_VDETECT
- R14 pad 1: Net-(U7-PA3) -> /STM/5V_VDETECT
- U7 pad 10: /12-5/5V_CURRENT_VOUT -> /12-5/5V_CURRENT_OCD
- U7 pad 11: /12-5/5V_CURRENT_VREF -> /12-5/5V_CURRENT_VOUT
- U7 pad 12: /12-5/5V_CURRENT_OCD -> /12-5/5V_CURRENT_VREF
- U7 pad 18: /48-12/12V_CURRENT_VOUT -> /STM_SDA
- U7 pad 19: /48-12/12V_CURRENT_VREF -> /STM_SCL
- U7 pad 20: /48-12/12V_CURRENT_OCD -> unconnected-(U7-PA10-Pad20)
- U7 pad 23: unconnected-(U7-PA13-Pad23) -> /STM/SYS_SWDIO
- U7 pad 24: unconnected-(U7-PA14-Pad24) -> /STM/SYS_SWCLK
- U7 pad 27: unconnected-(U7-PB4-Pad27) -> /STM/RPM_PG
- U7 pad 28: unconnected-(U7-PB5-Pad28) -> /STM/~{BMR_PG}
- U7 pad 29: unconnected-(U7-PB6-Pad29) -> /STM/~{BMR_SALERT}
- U7 pad 30: unconnected-(U7-PB7-Pad30) -> /STM/BMR_SDA
- U7 pad 31: unconnected-(U7-PB8-Pad31) -> /STM/BMR_SCL
- U7 pad 4: unconnected-(U7-PG10-Pad4) -> /STM/SYS_NRST
- U7 pad 5: unconnected-(U7-PA0-Pad5) -> /48-12/12V_CURRENT_VOUT
- U7 pad 6: unconnected-(U7-PA1-Pad6) -> /48-12/12V_CURRENT_VREF
- U7 pad 7: unconnected-(U7-PA2-Pad7) -> /STM/12V_VDETECT
- U7 pad 8: Net-(U7-PA3) -> /48-12/12V_CURRENT_OCD
- U7 pad 9: Net-(U7-PA4) -> /STM/5V_VDETECT

Commit message: update
Parts:
- removed C35, C36, C37: C_Small, Capacitor_SMD:C_0603_1608Metric
- removed the U3 at (213.1, 75.8)
- removed the U3 at (201.6, 79.7)
- removed U8: AZ1117-3.3, Package_TO_SOT_SMD:SOT-223-3_TabPin2
- added C20: 150pF 0Ohm, Capacitor_SMD:C_0603_1608Metric, F.Cu at (202.5, 103.0)
- added C27: C_Small, Capacitor_SMD:C_0603_1608Metric, F.Cu at (164.5, 103.5)
- added C30: 10uF, Capacitor_SMD:C_0603_1608Metric, F.Cu at (184.5, 90.8)
- added C31: 10uF, Capacitor_SMD:C_0603_1608Metric, F.Cu at (186.2, 94.0)
- added C34: 10uF, Capacitor_SMD:C_0603_1608Metric, F.Cu at (168.1, 106.3)
- added D1: 48V (BLUE), LED_SMD:LED_0603_1608Metric, F.Cu at (138.5, 103.5)
- added D2: 12V (RED), LED_SMD:LED_0603_1608Metric, F.Cu at (136.8, 103.5)
- added D3: 5V (GREEN), LED_SMD:LED_0603_1608Metric, F.Cu at (135.0, 103.5)
- added D4: 3V3 (PURPLE), LED_SMD:LED_0603_1608Metric, F.Cu at (133.2, 103.5)
- added D5: 12V_PG (RED), LED_SMD:LED_0603_1608Metric, F.Cu at (148.7, 103.2)
- added D6: 5V_PG (GREEN), LED_SMD:LED_0603_1608Metric, F.Cu at (147.0, 103.2)
- added J3: misc. power output, Connector_PinHeader_2.54mm:PinHeader_1x02_P2.54mm_Vertical, F.Cu at (244.9, 100.0)
- added J4: misc. power output, Connector_PinHeader_2.54mm:PinHeader_1x02_P2.54mm_Vertical, F.Cu at (239.3, 56.3)
- added J5: misc. power output, Connector_PinHeader_2.54mm:PinHeader_1x02_P2.54mm_Vertical, F.Cu at (234.8, 56.3)
- added J6: 796636-6, power_symbols:796636-6, F.Cu at (86.6, 140.8)
- added J7: I2C, Connector_PinHeader_2.54mm:PinHeader_1x03_P2.54mm_Vertical, F.Cu at (237.9, 111.0)
- added J8: SWD, Connector_PinHeader_2.54mm:PinHeader_1x05_P2.54mm_Vertical, F.Cu at (146.1, 91.8)
- added J9: BMR_I2C, Connector_PinHeader_2.54mm:PinHeader_1x03_P2.54mm_Vertical, F.Cu at (158.3, 85.0)
- added L1: 3u3 8.6mOhm, power_symbols:WE-MXGI_5030, F.Cu at (209.4, 95.4)
- added R15: 15k, Resistor_SMD:R_0603_1608Metric, F.Cu at (160.0, 108.0)
- added R16: 680R 1/4W 0603, Resistor_SMD:R_0603_1608Metric, F.Cu at (138.5, 100.2)
- added R17: 500R, Resistor_SMD:R_0603_1608Metric, F.Cu at (136.8, 100.2)
- added R18: 120R, Resistor_SMD:R_0603_1608Metric, F.Cu at (135.0, 100.2)
- added R19: 120R, Resistor_SMD:R_0603_1608Metric, F.Cu at (148.8, 100.2)
- added R20: 120R, Resistor_SMD:R_0603_1608Metric, F.Cu at (147.0, 100.2)
- added R21: 680R 1/4W 0603, Resistor_SMD:R_0603_1608Metric, F.Cu at (140.2, 100.2)
- added R22: 680R 1/4W 0603, Resistor_SMD:R_0603_1608Metric, F.Cu at (142.0, 100.2)
- added R23: 680R 1/4W 0603, Resistor_SMD:R_0603_1608Metric, F.Cu at (143.8, 100.2)
- added SW1: SW_Push, power_symbols:TS04-66-70-BK-160-SMT, F.Cu at (153.9, 95.5)
- added TP5V_CURRENT_VOUT1: TestPoint, TestPoint:TestPoint_THTPad_2.5x2.5mm_Drill1.2mm, F.Cu at (203.2, 111.5)
- added TP_12V_CURRENT_VOUT1: TestPoint, TestPoint:TestPoint_THTPad_2.5x2.5mm_Drill1.2mm, F.Cu at (192.5, 93.5)
- added TP_12V_OCD1: TestPoint, TestPoint:TestPoint_THTPad_2.5x2.5mm_Drill1.2mm, F.Cu at (208.8, 86.5)
- added TP_12V_PG1: TestPoint, TestPoint:TestPoint_THTPad_2.5x2.5mm_Drill1.2mm, F.Cu at (131.8, 90.2)
- added TP_12V_VDETECT1: TestPoint, TestPoint:TestPoint_THTPad_2.5x2.5mm_Drill1.2mm, F.Cu at (154.5, 109.0)
- added TP_1V1: TestPoint, TestPoint:TestPoint_THTPad_2.5x2.5mm_Drill1.2mm, F.Cu at (198.2, 111.5)
- added TP_3V1: TestPoint, TestPoint:TestPoint_THTPad_2.5x2.5mm_Drill1.2mm, F.Cu at (170.5, 91.5)
- added TP_5V_OCD1: TestPoint, TestPoint:TestPoint_THTPad_2.5x2.5mm_Drill1.2mm, F.Cu at (232.8, 112.0)
- added TP_5V_PG1: TestPoint, TestPoint:TestPoint_THTPad_2.5x2.5mm_Drill1.2mm, F.Cu at (211.5, 110.2)
- added TP_5V_VDETECT1: TestPoint, TestPoint:TestPoint_THTPad_2.5x2.5mm_Drill1.2mm, F.Cu at (166.5, 111.0)
- added U3: TPS56A37RPAR, power_symbols:TPS56A37RPAR, F.Cu at (203.1, 97.8)
- C11: value C_Small -> C_Polarized_Small; footprint Capacitor_SMD:C_0603_1608Metric -> Capacitor_THT:CP_Radial_D10.0mm_P5.00mm
- C13: value C_Polarized_Small -> C_Small; footprint Capacitor_THT:CP_Radial_D10.0mm_P5.00mm -> Capacitor_SMD:C_0603_1608Metric
- C19: value C_Small -> 100nF 1mOhm
- C21, C22: value 10uF -> 22uF 2.582mOhm
- C23: value 100nF -> 10uF 2.818mOhm
- C24: value C_Polarized_Small -> 10uF 2.818mOhm; footprint Capacitor_THT:CP_Radial_D10.0mm_P5.00mm -> Capacitor_SMD:C_0603_1608Metric
- C25: value 100nF -> 1uF 5mOhm
- C26: value C_Polarized_Small -> 22nF 1mOhm; footprint Capacitor_THT:CP_Radial_D10.0mm_P5.00mm -> Capacitor_SMD:C_0603_1608Metric
- C32: value C_Small -> 3u3
- C33: value C_Small -> 10uF
- J2: value 796636-6 -> misc. power output; footprint power_symbols:796636-6 -> Connector_PinHeader_2.54mm:PinHeader_1x02_P2.54mm_Vertical
- R1, R10, R6, R9: value 22k -> 10k
- R11: value 30k -> 10k
- R12: value 10k -> 30k
- R14: value 15k -> 10k
- R2, R7: value 4k7 -> 10k
- R3: value 100k -> 10k
- R4: value 10k -> 73k2
- R5: value 10k -> 100k
- R8: value 100k -> 52k3
- U1: value BMR4800116/005 -> MPQ1500-12V125-L48NBMC
- U2: footprint custom:LEM_HO150-NP -> power_symbols:LEM_HO150-NP
- U4: value RPM5.0-6.0 -> HO15-NP; footprint power_symbols:RPM5.0-6.0 -> Sensor_Current:LEM_HO8-NP
- U5: value HO8-NP -> TPS7A24125DBVR; footprint Sensor_Current:LEM_HO8-NP -> Package_TO_SOT_SMD:SOT-23-5
- U6: value AZ431LANTR-G1 -> TPS7A2433DBVR
- moved H2 166.3 mm to (260.8, 143.5)
- moved J2 133.4 mm to (240.3, 100.0), turned to 0 degrees
- moved H3 117.7 mm to (244.4, 89.9)
- moved G1 112.0 mm to (136.8, 131.2)
- moved C11 103.3 mm to (224.2, 57.5), turned to 90 degrees
- moved C32 95.1 mm to (152.2, 103.0), turned to 180 degrees
- moved C29 85.5 mm to (158.2, 92.4)
- moved R4 84.7 mm to (204.8, 102.2), turned to -90 degrees
- moved R5 83.3 mm to (206.2, 102.2), turned to -90 degrees
- moved C33 79.4 mm to (170.6, 103.8), turned to 180 degrees
- moved R9 78.5 mm to (155.2, 102.2), turned to 0 degrees
- moved C3 76.8 mm to (96.8, 70.0), turned to 0 degrees
- moved C28 74.3 mm to (167.8, 102.5), turned to -90 degrees
- moved C2 72.4 mm to (95.8, 123.8), turned to 0 degrees
- moved C19 67.7 mm to (204.5, 94.5)
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Connections:
- C11 pad 1: +48V -> +12V
- C11 pad 2: 48V_GND -> 12V_GND
- C19 pad 1: +12V -> Net-(U3-BOOT)
- C19 pad 2: 12V_GND -> Net-(U3-SW)
- C21 pad 1: +5V -> /12-5/5V_PRESENSE
- C22 pad 1: +3V3 -> /12-5/5V_PRESENSE
- C23 pad 1: +5V -> +12V
- C24 pad 1: +5V -> +12V
- C25 pad 1: +3V3 -> +12V
- C26 pad 1: +5V -> Net-(U3-SS)
- C28 pad 1: +5V -> +3V3
- C29 pad 1: +5V -> +3V3
- C32 pad 1: +5V -> /STM/SYS_NRST
- C33 pad 1: +5V -> +3V3
- J1 pad 13: +48V -> unconnected-(J1-Pad13)
- J1 pad 14: +48V -> unconnected-(J1-Pad14)
- J1 pad 15: 48V_GND -> unconnected-(J1-Pad15)
- J1 pad 16: 48V_GND -> unconnected-(J1-Pad16)
- J1 pad 21: +48V -> unconnected-(J1-Pad21)
- J1 pad 22: +48V -> unconnected-(J1-Pad22)
- J1 pad 23: 48V_GND -> unconnected-(J1-Pad23)
- J1 pad 24: 48V_GND -> unconnected-(J1-Pad24)
- J2 pad 1: +48V -> +5V
- J2 pad 2: +48V -> 12V_GND
- R1 pad 1: /48-12/12V_CURRENT_VREF -> +5V
- R1 pad 2: +5V -> /48-12/12V_CURRENT_OCD
- R10 pad 1: /48-12/5V_PRESENSE -> +3V3
- R10 pad 2: /48-12/12V_CURRENT_OCD -> /STM_SDA
- R11 pad 1: /48-12/12V_PRESENSE -> +3V3
- R11 pad 2: /STM/12V_VDETECT -> /STM_SCL
- R12 pad 1: /STM/12V_VDETECT -> /48-12/12V_PRESENSE
- R12 pad 2: 12V_GND -> /STM/12V_VDETECT
- R13 pad 1: /12-5/5V_PRESENSE -> /STM/12V_VDETECT
- R13 pad 2: /STM/5V_VDETECT -> 12V_GND
- R14 pad 1: /STM/5V_VDETECT -> /12-5/5V_PRESENSE
- R14 pad 2: 12V_GND -> /STM/5V_VDETECT
- R2 pad 1: /48-12/12V_CURRENT_VREF -> Net-(U1-SA1)
- R2 pad 2: Net-(U3-REF) -> 12V_GND
- R3 pad 1: Net-(U3-REF) -> Net-(U1-SA0)
- R4 pad 1: Net-(U1-SA1) -> /12-5/5V_PRESENSE
- R4 pad 2: 12V_GND -> Net-(U3-FB)
- R5 pad 1: Net-(U1-SA0) -> /12-5/5V_PRESENSE
- R5 pad 2: 12V_GND -> 5V_PG
- R6 pad 1: /12-5/5V_PRESENSE -> +5V
- R6 pad 2: /12-5/5V_CURRENT_VREF -> /12-5/5V_CURRENT_OCD
- R7 pad 1: /12-5/5V_CURRENT_VREF -> Net-(U3-FB)
- R7 pad 2: Net-(U6-REF) -> 12V_GND
- R8 pad 1: Net-(U6-REF) -> Net-(U3-MODE)
- R9 pad 1: /12-5/5V_PRESENSE -> +3V3
- R9 pad 2: /12-5/5V_CURRENT_OCD -> /STM/SYS_NRST
- U1 pad 11: /48-12/BMR_SDA -> BMR_SDA
- U1 pad 12: /48-12/~{BMR_SALERT} -> ~{BMR_SALERT}
- U1 pad 13: /48-12/BMR_SCL -> BMR_SCL
- U1 pad 6: /48-12/~{BMR_PG} -> ~{BMR_PG}
- U2 pad 4: /48-12/12V_CURRENT_VREF -> +1V25
- U5 pad 1: /12-5/5V_PRESENSE -> +5V
- U5 pad 3: /12-5/5V_CURRENT_VOUT -> +5V
- U5 pad 4: /12-5/5V_CURRENT_VREF -> unconnected-(U5-FB-Pad4)
- U5 pad 5: /12-5/5V_CURRENT_OCD -> +1V25
- U6 pad 1: (no net) -> +5V
- U6 pad 2: (no net) -> 12V_GND
- U6 pad 3: /12-5/5V_CURRENT_VREF -> +5V
- U6 pad 4: Net-(U6-REF) -> unconnected-(U6-FB-Pad4)
- U6 pad 5: 12V_GND -> +3V3
- U7 pad 12: /12-5/5V_CURRENT_VREF -> +1V25
- U7 pad 27: /STM/RPM_PG -> 5V_PG
- U7 pad 28: /STM/~{BMR_PG} -> ~{BMR_PG}
- U7 pad 29: /STM/~{BMR_SALERT} -> ~{BMR_SALERT}
- U7 pad 30: /STM/BMR_SDA -> BMR_SDA
- U7 pad 31: /STM/BMR_SCL -> BMR_SCL
- U7 pad 6: /48-12/12V_CURRENT_VREF -> +1V25
Routing:
- net +5V: track 0.00 -> 206.0 mm, vias 0 -> 10
- net +1V25: track 0.00 -> 169.1 mm, vias 0 -> 5
- net 12V_GND: track 25.7 -> 184.5 mm, vias 3 -> 243
- net /STM_SCL: track 0.00 -> 145.9 mm, vias 0 -> 2
- net /STM_SDA: track 0.00 -> 139.6 mm, vias 0 -> 3
- net 5V_PG: track 0.00 -> 126.4 mm, vias 0 -> 5
- net +3V3: track 0.00 -> 106.2 mm, vias 0 -> 8
- net ~{BMR_PG}: track 0.00 -> 101.8 mm, vias 0 -> 3
- net +12V: track 0.00 -> 86.0 mm, vias 0 -> 94
- net /48-12/12V_CURRENT_OCD: track 0.00 -> 82.7 mm, vias 0 -> 3
- net /12-5/5V_CURRENT_OCD: track 10.0 -> 87.3 mm
- net +48V: track 135.1 -> 59.7 mm, vias 0 -> 135
- net 48V_GND: track 124.8 -> 49.5 mm, vias 6 -> 71
- net /12-5/5V_CURRENT_VOUT: track 9.11 -> 81.3 mm
- net /48-12/12V_PRESENSE: track 0.00 -> 70.0 mm, vias 0 -> 1
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- added copper zone on B.Cu, net +12V
- added copper zone on B.Cu, net +48V
- added copper zone on B.Cu, net +5V
- added copper zone on B.Cu, net /48-12/12V_PRESENSE
- added copper zone on F.Cu, net 48V_GND
- added copper zone on F.Cu, net Net-(U3-SW)
Other:
- board size 165.1 x 98.5 mm -> 186 x 111.2 mm
- board text added: "12V"
- board text added: "3V3"
- board text added: "48V"
- board text added: "5V"
- board text added: "BUS"
- board text added: "PG"
- board text added: "SDA SCL GND"
- board text added: "Test Bench Power Slab v0.1 Sam Nadol"

Commit message: final
Parts:
- added G***: LOGO, LOGO, F.Cu at (237.8, 132.0)
- added R12: 0R, Resistor_SMD:R_0603_1608Metric, F.Cu at (172.0, 100.2)
- added R13: 0R, Resistor_SMD:R_0603_1608Metric, F.Cu at (172.0, 98.7)
- C1, C2: value C_Polarized_Small -> 330uF 63V poly; footprint Capacitor_THT:CP_Radial_D18.0mm_P7.50mm -> Capacitor_THT:CP_Radial_D12.5mm_P5.00mm
- C10: value C_Small -> 0.1uF 63V
- C11, C12: value C_Polarized_Small -> 2.2mF 16V poly; footprint Capacitor_THT:CP_Radial_D10.0mm_P5.00mm -> Capacitor_THT:CP_Radial_D18.0mm_P7.50mm
- C13, C14, C15, C16, C17, C18: value C_Small -> 10uF
- C27: value C_Small -> 0.1uF
- C28, C29: value C_Small -> 1uF
- C3, C4, C5: value C_Polarized_Small -> 100uF 63V poly; footprint Capacitor_THT:CP_Radial_D8.0mm_P5.00mm -> Capacitor_THT:CP_Radial_D8.0mm_P3.50mm
- C6, C7, C8, C9: value C_Small -> 10uF 63V
- J2, J3, J4, J5: value misc. power output -> 2.54mm header
- R18: renamed from R16; value 680R 1/4W 0603 -> 680R 1/4W
- R19: renamed from R17; value 500R -> 680R 1/4W
- R23: renamed from R21; value 680R 1/4W 0603 -> 680R 1/4W
- R24: renamed from R22; value 680R 1/4W 0603 -> 680R 1/4W
- R25: renamed from R23; value 680R 1/4W 0603 -> 680R 1/4W
- moved J5 26.2 mm to (235.0, 82.5), turned to 0 degrees
- moved J4 26.2 mm to (240.0, 82.5), turned to 0 degrees
- moved C11 12.5 mm to (236.8, 58.5)
- moved C18 7.97 mm to (249.5, 72.8), turned to 90 degrees
- moved C16 6.81 mm to (244.5, 72.8), turned to 90 degrees
- moved C14 6.68 mm to (242.0, 68.0)
- moved C15 6.68 mm to (242.0, 65.5)
- moved C13 6.68 mm to (242.0, 70.5)
- moved C2 6.61 mm to (96.7, 117.2)
- moved C17 6.51 mm to (247.0, 72.8), turned to 90 degrees
- moved C12 4.39 mm to (217.0, 58.5)
- moved R10 3.26 mm to (174.2, 96.5)
- moved R11 3.01 mm to (175.8, 96.5)
- moved C1 2.20 mm to (96.7, 102.2)
- moved C3 0.96 mm to (97.3, 70.8)
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- renumbered J9 to J7, J7 to J8, J8 to J9, R12 to R14, R13 to R15, R14 to R16, R15 to R17, R18 to R20, R19 to R21, R20 to R22, TP_1V1 to TP_1V25_1, TP_3V1 to TP_3V_1
Connections:
- J1 pad 01: unconnected-(J1-Pad01) -> 12V_GND
- J1 pad 02: unconnected-(J1-Pad02) -> 12V_GND
- J1 pad 03: unconnected-(J1-Pad03) -> +5V
- J1 pad 04: unconnected-(J1-Pad04) -> +5V
- U7 pad 18: /STM_SDA -> Net-(U7-PA8)
- U7 pad 19: /STM_SCL -> Net-(U7-PA9)
Routing:
- net 12V_GND: track 184.5 -> 231.7 mm, vias 243 -> 242
- net +12V: track 86.0 -> 96.9 mm, vias 94 -> 92
- net +48V: track 59.7 -> 67.0 mm, vias 135 -> 140
- net 48V_GND: track 49.5 -> 56.6 mm, vias 71 -> 76
- net /STM_SDA: track 139.6 -> 132.6 mm
- net /STM_SCL: track 145.9 -> 141.3 mm
- net Net-(U7-PA8): track 0.00 -> 4.31 mm
- net Net-(U7-PA9): track 0.00 -> 4.00 mm
- net +3V3: track 106.2 -> 108.5 mm
Other:
- board text added: "12V GND"
- board text added: "5V GND"
- board text added: "GND BMR_SCL BMR_SDA"
- board text added: "GND ~{RST} CLK DIO 3V3"
- board text added: "JLCJLCJLCJLC"
- board text added: "OUTPUT"
- board text added: "RESET"
- board text added: "TETHER"
- board text added: "X18 Test Bench Power Slab v0.1 Sam Nadol Leads: Sahil, Keona, Nicholas"
- board text removed: "Test Bench Power Slab v0.1 Sam Nadol"
