File: power/power.kicad_sch (KiCad schematic)
At the start: 2 parts, among them J1 ET60T-D04-3-08-D04-X-R1-S, J2 796636-6

Commit message: work
Parts:
- added C1, C12, C13, C2: C_Polarized_Small, Capacitor_THT:CP_Radial_D18.0mm_P7.50mm, symbol Device:C_Polarized_Small
- added C10, C11, C20, C21, C22, C23, C24, C25, C26, C27, C28, C29, C34, C35, C36, C37, C38, C39, C40, C6, C7, C8, C9: C_Small, Capacitor_SMD:C_0603_1608Metric, symbol Device:C_Small
- added C14, C15, C16, C17, C18, C19, C30, C31, C32, C33: C_Polarized_Small, Capacitor_THT:CP_Radial_D10.0mm_P5.00mm, symbol Device:C_Polarized_Small
- added C3, C4, C5: C_Polarized_Small, Capacitor_THT:CP_Radial_D8.0mm_P5.00mm, symbol Device:C_Polarized_Small
- added G1: LOGO, custom:logo, symbol custom:LOGO
- added R1: 10k, Resistor_SMD:R_0603_1608Metric, symbol Device:R_Small
- added U1: BMR4912510/871, power_symbols:BMR491_FPM, symbol power_symbols:BMR4912510_871
- added U2: RPM5.0-6.0, power_symbols:RPM5.0-6.0, symbol power_symbols:RPM5.0-6.0
Connections:
- net 5V_GND is gone; now on net 12V_GND: J1.09, J1.10, J1.17, J1.18
- net +12V: now also C12.1, C13.1, C14.1, C15.1, C16.1, C17.1, C18.1, C19.1, C20.1, C21.1, C22.1, C23.1, C24.1, C25.1, C26.1, C27.1, C28.1, C29.1, U1.15 (+SENSE), U1.7 (+OUT), U1.8 (+OUT), U2.A1 (VIN), U2.A2 (VIN)
- net +48V: now also C1.1, C10.1, C11.1, C2.1, C3.1, C4.1, C5.1, C6.1, C7.1, C8.1, C9.1, U1.1 (+IN)
- net +5V: now also C30.1, C31.1, C32.1, C33.1, C34.1, C35.1, C36.1, C37.1, C38.1, C39.1, C40.1, U2.A5 (VOUT), U2.B5 (VOUT), U2.C5 (SENSE)
- net 12V_GND: now also C12.2, C13.2, C14.2, C15.2, C16.2, C17.2, C18.2, C19.2, C20.2, C21.2, C22.2, C23.2, C24.2, C25.2, C26.2, C27.2, C28.2, C29.2, C30.2, C31.2, C32.2, C33.2, C34.2, C35.2, C36.2, C37.2, C38.2, C39.2, C40.2, R1.2, U1.10 (-SENSE), U1.4 (-OUT), U1.5 (-OUT), U2.A3 (GND), U2.A4 (GND), U2.B1 (GND), U2.B2 (GND), U2.B3 (GND), U2.B4 (GND), U2.C2 (GND), U2.C3 (GND), U2.C4 (GND), U2.D2 (GND), U2.D3 (GND), U2.D4 (GND), U2.D5 (GND), U2.E3 (GND), U2.E4 (GND)
- net 48V_GND: now also C1.2, C10.2, C11.2, C2.2, C3.2, C4.2, C5.2, C6.2, C7.2, C8.2, C9.2, U1.2 (RC), U1.3 (-IN)
- net RPM_PG: now reaches J1.04
- net RPM_PG: now also U2.D1 (PGOOD)
- net BMR_PG: now reaches J1.05
- net BMR_PG: now also U1.9 (CTRL)
- net BMR_SDA: now reaches J1.06
- net BMR_SDA: now also U1.11 (SDA)
- net BMR_SCL: now reaches J1.07
- net BMR_SCL: now also U1.13 (SCL)
- net BMR_SALERT: now reaches J1.08
- net BMR_SALERT: now also U1.12 (SALERT)
- new net: R1.1, U1.14 (SA1)
- no-connect marks 48 -> 46
Other:
- note added: "12-05V OUTPUT CAPS"
- note added: "48-12V INPUT CAPS"
- note added: "48-12V OUTPUT 12-05V INPUT CAPS"
- note added: "HF decoupling 10uF 10V MLCC"
- note added: "HF decoupling 10uF 16V MLCC"
- note added: "HF decoupling 10uF 63V MLCC"
- note added: "VHF decoupling 0.1uF 10V MLCC"
- note added: "VHF decoupling 0.1uF 63V MLCC"
- note added: "bulk storage 10mF 16V poly"
- note added: "bulk storage 2.2mF 10V poly"
- note added: "bulk storage 330uF 63V poly"
- note added: "medium storage 100uF 63V poly"
- note added: "medium storage 2.2mF 16V poly"
- note added: "medium storage 470uF 10V poly"
- moved on the sheet: J1, J2

Commit message: stuff
Parts:
- removed C12, C13: C_Polarized_Small, Capacitor_THT:CP_Radial_D18.0mm_P7.50mm, symbol Device:C_Polarized_Small
- removed C16, C17, C18, C19: C_Polarized_Small, Capacitor_THT:CP_Radial_D10.0mm_P5.00mm, symbol Device:C_Polarized_Small
- removed U1: BMR4912510/871, power_symbols:BMR491_FPM, symbol power_symbols:BMR4912510_871
- added H1, H2, H3: MountingHole, MountingHole:MountingHole_3.2mm_M3, symbol Mechanical:MountingHole
- added R2: 10k, Resistor_SMD:R_0603_1608Metric, symbol Device:R_Small
- added U1: STM32F091CCTx, Package_QFP:LQFP-48_7x7mm_P0.5mm, symbol MCU_ST_STM32F0:STM32F091CCTx
- added U3: BMR4800116/005, power_symbols:BMR491_FPM, symbol power_symbols:BMR4800116/005
Connections:
- net +12V: now also U3.7 (+OUT), U3.8 (+OUT)
- net +48V: now also U3.1 (+IN)
- net 12V_GND: now also R2.2, U3.10 (DGND), U3.4 (-OUT), U3.5 (-OUT), U3.9 (CTRL)
- net 48V_GND: now also U3.2 (RC), U3.3 (-IN)
- net BMR_SCL: now also U3.13 (SCL)
- net BMR_SDA: now also U3.11 (SDA)
- net at R1.1: now also U3.15 (SA0)
- net BMR_PG renamed ~{BMR_PG}
- net ~{BMR_PG}: now also U3.6 (PG)
- net BMR_SALERT renamed ~{BMR_SALERT}
- net ~{BMR_SALERT}: now also U3.12 (SALERT)
- new net: R2.1, U3.14 (SA1)
- new net: U1.23 (VSS), U1.35 (VSS), U1.47 (VSS)
Other:
- note removed: "bulk storage 10mF 16V poly"
- moved on the sheet: C14, C15, R1

Commit message: update
Parts:
- removed C14, C15, C30, C31, C32, C33: C_Polarized_Small, Capacitor_THT:CP_Radial_D10.0mm_P5.00mm, symbol Device:C_Polarized_Small
- removed C20, C21, C22, C23, C24, C25, C26, C27, C28, C29, C34, C35, C36, C37, C38, C39, C40: C_Small, Capacitor_SMD:C_0603_1608Metric, symbol Device:C_Small
- removed U1: STM32F091CCTx, Package_QFP:LQFP-48_7x7mm_P0.5mm, symbol MCU_ST_STM32F0:STM32F091CCTx
- removed U2: RPM5.0-6.0, power_symbols:RPM5.0-6.0, symbol power_symbols:RPM5.0-6.0
- removed U3: BMR4800116/005, power_symbols:BMR491_FPM, symbol power_symbols:BMR4800116/005
- added D1: 48V (BLUE), symbol Device:LED
- added D2: 5V (GREEN), symbol Device:LED
- added D3: 12V (RED), symbol Device:LED
- added D4: 5V_PG (GREEN), symbol Device:LED
- added D5: 12V_PG (RED), symbol Device:LED
- added J3, J4, J5, J7: misc. power output, symbol Connector:Conn_01x02_Pin
- added R16: 1k2 1W, symbol Device:R_Small
- added R17, R3: 120R, symbol Device:R_Small
- added R18: 500R, symbol Device:R_Small
- R1: value 10k -> 1k2 1W; footprint Resistor_SMD:R_0603_1608Metric -> (none)
- R2: value 10k -> 120R; footprint Resistor_SMD:R_0603_1608Metric -> (none)
Connections:
- net +12V: now also D3.2 (A), J3.1 (Pin_1), J4.1 (Pin_1)
- net +48V: now also D1.2 (A)
- net +5V: now also D2.2 (A), D5.2 (A), J5.1 (Pin_1), J7.1 (Pin_1)
- net 12V_GND: no longer J1.09, J1.10, J1.17, J1.18, R1.2, R2.2
- net 48V_GND: now also R1.2
- net RPM_PG: now also D4.2 (A); no longer J1.04
- net ~{BMR_PG}: now also R2.2; no longer J1.05
- net at R2.1: now also D5.1 (K)
- net at R1.1: now also R16.2
- net BMR_SCL renamed STM_SDA
- net BMR_SDA: no longer names the net of J1.06
- net ~{BMR_SALERT} renamed STM_SCL
- new net: D3.1 (K), R18.1
- new net: D4.1 (K), R3.1
- new net: D2.1 (K), R17.1
- new net: D1.1 (K), R16.1
- new net 5V_GND: J1.09, J1.10, J1.17, J1.18, J3.2 (Pin_2), J4.2 (Pin_2), J5.2 (Pin_2), J7.2 (Pin_2), R17.2, R18.2, R3.2
Other:
- added sheet 12-5 (12-5.kicad_sch)
- added sheet 48-12 (48-12.kicad_sch)
- added sheet STM (STM.kicad_sch)
- note removed: "12-05V OUTPUT CAPS"
- note removed: "48-12V OUTPUT 12-05V INPUT CAPS"
- note removed: "HF decoupling 10uF 10V MLCC"
- note removed: "HF decoupling 10uF 16V MLCC"
- note removed: "VHF decoupling 0.1uF 10V MLCC"
- note removed: "bulk storage 2.2mF 10V poly"
- note removed: "medium storage 2.2mF 16V poly"
- note removed: "medium storage 470uF 10V poly"
- moved on the sheet: C1, C10, C11, C2, C3, C4, C5, C6, C7, C8, C9, J2

Commit message: work
Parts:
- removed D1: 48V (BLUE), symbol Device:LED
- removed D2: 5V (GREEN), symbol Device:LED
- removed D3: 12V (RED), symbol Device:LED
- removed D4: 5V_PG (GREEN), symbol Device:LED
- removed D5: 12V_PG (RED), symbol Device:LED
- removed R1, R16: 1k2 1W, symbol Device:R_Small
- removed R17, R2, R3: 120R, symbol Device:R_Small
- removed R18: 500R, symbol Device:R_Small
Other:
- sheet 12-5 ports: added none; removed 5V_CURRENT_VREF
- sheet 48-12 ports: added none; removed 12V_CURRENT_VREF
- sheet STM ports: added none; removed 12V_CURRENT_VREF, 5V_CURRENT_VREF
- moved on the sheet: J2, J3, J4, J5, J7

Commit message: update
Parts:
- removed C11: C_Small, Capacitor_SMD:C_0603_1608Metric, symbol Device:C_Small
- J2: renamed from J5; footprint (none) -> Connector_PinHeader_2.54mm:PinHeader_1x02_P2.54mm_Vertical
- J3: renamed from J7; footprint (none) -> Connector_PinHeader_2.54mm:PinHeader_1x02_P2.54mm_Vertical
- J4: renamed from J3; footprint (none) -> Connector_PinHeader_2.54mm:PinHeader_1x02_P2.54mm_Vertical
- J5: renamed from J4; footprint (none) -> Connector_PinHeader_2.54mm:PinHeader_1x02_P2.54mm_Vertical
- renumbered J2 to J6
Connections:
- net +48V: no longer J1.13, J1.14, J1.21, J1.22
- net 48V_GND: no longer J1.15, J1.16, J1.23, J1.24

Commit message: final
Parts:
- C1, C2: value C_Polarized_Small -> 330uF 63V poly; footprint Capacitor_THT:CP_Radial_D18.0mm_P7.50mm -> Capacitor_THT:CP_Radial_D12.5mm_P5.00mm; LCSC (none) -> C437640; MPN (none) -> 63YXJ330M12.5X20
- C10: value C_Small -> 0.1uF 63V; now not fitted
- C3, C4, C5: value C_Polarized_Small -> 100uF 63V poly; footprint Capacitor_THT:CP_Radial_D8.0mm_P5.00mm -> Capacitor_THT:CP_Radial_D8.0mm_P3.50mm; LCSC (none) -> C134638; MPN (none) -> RXW101M1JBK-0815
- C6, C7, C8, C9: value C_Small -> 10uF 63V; now not fitted
- G1, H1, H2, H3: MPN (none) -> -
- J1: MANUFACTURER Samtec -> (none); MAXIMUM_PACKAGE_HEIGHT 10.0 mm -> (none); MPN (none) -> -; PARTREV J -> (none); STANDARD Manufacturer Recommendations -> (none)
- J2, J3, J4, J5: value misc. power output -> 2.54mm header; MPN (none) -> -
- J6: MPN (none) -> 796636-6
Connections:
- net +5V: now also J1.03, J1.04
- net 5V_GND: now also J1.01, J1.02
- no-connect marks 46 -> 50
