File: MCU and Pi Board/mcu and pi board/mcu and pi board.kicad_pcb (KiCad board)
At the start: 4 copper layers, 143.6 x 215.8 mm, 112 parts, among them IC3 CSD17578Q3A, IC4 CSD17578Q3A, J1 PJ-002A, J10 ET60T-D04-0-00-D04-X-R1-S, J12 430450428, J13 IPBT-105-H1-T-D-GP, J14 IPBT-105-H1-T-D-GP, J15 Conn_01x28_Socket, J16 Conn_01x28_Socket, J17 DebugnBoot, J18 UART-PINS, J19 Conn_01x02_Pin, J2 ET60S-D04-3-08-D04-X-R1-S, J20 Conn_01x03_Pin, J21 Conn_01x05, J22 Conn_01x03_Pin, J23 TB006-508-03BE, J24 TB006-508-03BE, J25 TB006-508-03BE, J26 Conn_01x03_Pin, J27 Conn_01x02_Pin, J28 Conn_02x04_Counter_Clockwise, J29 Conn_02x02_Pin, J3 BM04B-GHS-TBT, J30 Conn_01x04_Pin, J31 Conn_01x04_Pin, J32 Conn_01x02_Pin, J33 Conn_01x02_Pin, J34 Conn_01x03_Pin, J35 Conn_02x09_Counter_Clockwise, J4 PJ-002A, J5 Conn_01x03_Pin, J6 Conn_01x04_Socket, J7 Conn_01x04_Pin, J8 PWM Connector, J9 ESC ADAPTER - BACKPLANE, Q1 BSC010N04LS6ATMA1, Q2 BSC010N04LS6ATMA1, U1 STM32F091CCT6, U2 LM3940IMPX-3.3/NOPB, U3 LTC4370CMS_PBF, U4 TPS40305DRCR, U5 RASPBERRY_PI_4B_4GB, U6 MC74HC157ADR2G, U7 MC74HC157ADR2G

Commit message: basically done, added a bunch of vias for no reason, for love of the game
Parts:
- C19: value 0.1u -> 10u
- moved C18 16.1 mm to (181.6, 91.0)
- moved C19 15.9 mm to (181.6, 98.6)
Connections:
- J35 pad 1: /pi/TR03 -> /pi/TR01
- J35 pad 10: unconnected-(J35-Pin_10-Pad10) -> /pi/GPIO16
- J35 pad 11: /pi/TR02 -> /pi/GPIO5
- J35 pad 12: /pi/TR01 -> /pi/GPIO12
- J35 pad 13: /pi/TR00 -> /pi/ID_SD
- J35 pad 14: /pi/GPIO25 -> /pi/ID_SC
- J35 pad 15: /pi/GPIO24 -> /pi/CS_TOOLS
- J35 pad 16: /pi/ID_SC -> /pi/GPIO25
- J35 pad 17: /pi/ID_SD -> unconnected-(J35-Pin_17-Pad17)
- J35 pad 18: /pi/CS_TOOLS -> /pi/GPIO24
- J35 pad 2: /pi/GPIO5 -> /pi/TR00
- J35 pad 3: /pi/GPIO6 -> /pi/TR03
- J35 pad 4: /pi/GPIO12 -> /pi/TR02
- J35 pad 6: /pi/GPIO16 -> /pi/GPIO21
- J35 pad 9: /pi/GPIO21 -> /pi/GPIO6
Routing:
- net /pi/GPIO25: track 0.00 -> 81.5 mm
- net /pi/CS_TOOLS: track 37.1 -> 115.5 mm
- net /pi/ID_SD: track 0.00 -> 74.5 mm
- net /pi/ID_SC: track 0.00 -> 70.9 mm
- net /pi/GPIO5: track 0.00 -> 69.0 mm
- net /pi/GPIO6: track 0.00 -> 63.6 mm
- net /pi/GPIO12: track 0.00 -> 62.9 mm
- net /pi/GPIO13: track 0.00 -> 55.6 mm
- net /pi/GPIO16: track 0.00 -> 54.9 mm
- net /pi/GPIO19: track 0.00 -> 52.0 mm
- net /pi/GPIO20: track 0.00 -> 50.2 mm
- net /pi/GPIO22: track 0.00 -> 45.1 mm
- net /pi/GPIO21: track 0.00 -> 44.8 mm
- net /pi/GPIO23: track 0.00 -> 41.5 mm
- net /pi/GPIO27: track 0.00 -> 40.5 mm
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
Commit message: basically done
Parts:
- added TP2: TestPoint, TestPoint:TestPoint_Pad_D4.0mm, F.Cu at (231.0, 66.6)
- added TP6: TestPoint, TestPoint:TestPoint_Pad_D4.0mm, F.Cu at (198.1, 219.8)
- moved C31 14.3 mm to (242.9, 195.9), turned to 0 degrees
- moved C28 11.6 mm to (239.1, 195.3), turned to 90 degrees
- moved IC1 11.4 mm to (240.1, 199.2)
- moved C27 9.55 mm to (231.6, 200.9)
- moved R12 9.34 mm to (233.6, 197.9)
- moved C33 9.12 mm to (242.1, 202.3), turned to 0 degrees
- moved C30 8.00 mm to (242.5, 204.5), turned to 0 degrees
- moved C20 7.02 mm to (237.8, 189.8), turned to 90 degrees
- moved TP7 5.51 mm to (197.8, 227.9)
- moved R14 5.37 mm to (228.1, 200.7), turned to 0 degrees
- moved C26 4.76 mm to (238.7, 205.6)
- moved R13 4.68 mm to (239.4, 208.6), turned to 90 degrees
- moved C23 4.48 mm to (231.2, 203.7)
- moved IC2 3.70 mm to (234.6, 206.8), turned to 180 degrees
- moved R10 2.61 mm to (230.7, 196.8)
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- renumbered C3 to C1, C1 to C10, C2 to C11, C19 to C12, C18 to C13, C13 to C14, C11 to C15, C14 to C16, C15 to C17, C12 to C18, C16 to C19, C4 to C2, C31 to C20, C23 to C21, C24 to C22, C35 to C23, C34 to C24, C36 to C25, C33 to C26, C37 to C27, C8 to C29, C7 to C3, C29 to C31, C26 to C32, C32 to C33, C40 to C34, C25 to C35, C27 to C36, C39 to C37, C17 to C39, C6 to C4, C22 to C40, C21 to C6, C10 to C7, C20 to C8, D4 to D1, D1 to D2, D2 to D4, IC4 to IC1, IC3 to IC2, J3 to J1, J12 to J10, J31 to J11, J19 to J12, J34 to J13, J10 to J14, J16 to J15, J15 to J16, J27 to J17, J7 to J18, J20 to J19, J30 to J20, J33 to J21, J29 to J23, J13 to J24, J35 to J25, J17 to J27, J18 to J28, J5 to J29, J1 to J3, J8 to J30, J9 to J31, J23 to J32, J24 to J33, J25 to J34, J6 to J4, J4 to J5, J14 to J6, J28 to J7, J32 to J8, J21 to J9, L2 to L1, Q2 to Q1, Q1 to Q2, R8 to R1, R13 to R10, R15 to R12, R12 to R13, R4 to R15, R6 to R16, R5 to R2, R7 to R3, R3 to R4, R18 to R5, R19 to R6, R1 to R7, R2 to R8, R16 to R9, TP4 to TP3, TP3 to TP4, TP2 to TP7, U3 to U1, U1 to U3, U5 to U4, U6 to U5, U7 to U6, U4 to U7
Routing:
- net /power/servo power/SW : track 9.83 -> 25.2 mm, vias 0 -> 4
- net +12V: track 17.1 -> 6.47 mm
- net /power/servo power/HDRV: track 15.2 -> 5.23 mm, vias 2 -> 0
- net +6V: track 0.00 -> 9.81 mm
- net GND: track 135.8 -> 126.2 mm, vias 658 -> 60
- net /power/servo power/LDRV/OC: track 15.2 -> 6.16 mm, vias 2 -> 0
- net Net-(U4-EN/SS): track 6.47 -> 10.6 mm
- net /power/servo power/BP: track 8.45 -> 4.94 mm
- net Net-(U4-PGOOD): track 7.78 -> 4.65 mm, vias 0 -> 2
- net /power/servo power/BOOT: track 5.39 -> 2.55 mm
- net /power/servo power/FB: track 19.2 -> 16.8 mm
- net Net-(C36-Pad2): track 2.88 -> 5.10 mm
- net /power/servo power/COMP: track 9.39 -> 7.38 mm
- net /MCU/GPIO9: track 97.2 -> 99.1 mm
- net /MCU/GPIO8: track 17.2 -> 19.0 mm
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Other:
- board text added: "12V"
- board text added: "3.3V"
- board text added: "5V"
- board text added: "5V Out"
- board text added: "5V PWR IN"
- board text added: "6V"
- board text added: "CS"
- board text added: "CS_TOOLS"
- board text added: "ESC PWM Breakout"
- board text added: "ESC_0"
- board text added: "ESC_1"
- board text added: "ESC_2"
- board text added: "ESC_3"
- board text added: "GND"
- board text added: "GPIO05"
- board text added: "GPIO06"
- board text added: "GPIO12"
- board text added: "GPIO13"
- board text added: "GPIO14"
- board text added: "GPIO15"
- board text added: "GPIO16"
- board text added: "GPIO17"
- board text added: "GPIO18"
- board text added: "GPIO19"
- board text added: "GPIO20"
- board text added: "GPIO21"
- board text added: "GPIO22"
- board text added: "GPIO23"
- board text added: "GPIO24"
- board text added: "GPIO25"
- board text added: "GPIO27"
- board text added: "GPIO4"
- board text added: "I2C1 Breakout"
- board text added: "I2C2 Breakout"
- board text added: "ID_SC"
- board text added: "ID_SD"
- board text added: "MISO"
- board text added: "MOSI"
- board text added: "PA1"
- board text added: "PA11"
- board text added: "PA12"
- board text added: "PA15"
- board text added: "PB0"
- board text added: "PB2"
- board text added: "PB8"
- board text added: "PB9"
- board text added: "PWM 0"
- board text added: "PWM 1"
- board text added: "PWM 2"
- board text added: "PWM 3"
- board text added: "PWM 4"
- board text added: "Programming Header"
- board text added: "RP"
- board text added: "RX"
- board text added: "SCK"
- board text added: "SCL"
- board text added: "SCLK"
- board text added: "SDA"
- board text added: "SEL"
- board text added: "SERVO 0"
- board text added: "SERVO 1"
- board text added: "SERVO 2"
- board text added: "SPI1 Breakout"
- board text added: "SPI2 Breakout"
- board text added: "STM"
- board text added: "STM ESC PWM Breakout"
- board text added: "STM PWM Breakout"
- board text added: "STM_CS"
- board text added: "SWCLK"
- board text added: "SWDIO"
- board text added: "TR00"
- board text added: "TR01"
- board text added: "TR02"
- board text added: "TR03"
- board text added: "TX"
- board text added: "Telemetry"

Commit message: added names and pete
Parts:
- added G***: LOGO, LOGO, F.Cu at (174.4, 215.0)
Other:
- board text added: "Made by Aman Katyal Leads: Vijay, Keona, Sahil"
