File: MCU and Pi Board/mcu and pi board/sensors.kicad_sch (KiCad schematic)
At the start: 2 parts, among them J3 BM04B-GHS-TBT, J6 Conn_01x04_Socket

Commit message: added some testpoints and some labeling
Other:
- note added: "have onboard 10k pullup resistors"
Changed lines of the file:
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@@
+		)
+	)
+	(text "have onboard 10k pullup resistors\n"
+		(exclude_from_sim no)
+		(at 148.59 46.228 0)
+		(effects
+			(font
+				(size 1.27 1.27)
+			)
 		)
 	)

Commit message: minor edits
Changed lines of the file:
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@@
 	(text "have onboard 10k pullup resistors\n"
 		(exclude_from_sim no)
-		(at 148.59 46.228 0)
+		(at 147.828 46.99 0)
 		(effects
 			(font

Commit message: pretty much done i think
Other:
- moved on the sheet: J3
Changed lines of the file:
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@@
 	(text "Bar High-Resolution Depth/Pressure Sensors \nAddress is 0x76\n"
 		(exclude_from_sim no)
-		(at 101.6 70.358 0)
+		(at 134.62 62.738 0)
 		(effects
 			(font
@@
 	(hierarchical_label "SCL"
 		(shape input)
-		(at 93.98 77.47 180)
+		(at 127 69.85 180)
 		(effects
 			(font
@@
 	(hierarchical_label "SDA"
 		(shape input)
-		(at 93.98 80.01 180)
+		(at 127 72.39 180)
 		(effects
 			(font
@@
 	(symbol
 		(lib_id "power:GND")
-		(at 93.98 82.55 270)
+		(at 127 74.93 270)
 		(unit 1)
 		(exclude_from_sim no)
@@
 		(fields_autoplaced yes)
 		(property "Reference" "#PWR016"
-			(at 87.63 82.55 0)
+			(at 120.65 74.93 0)
 			(effects
 				(font
@@
 		)
 		(property "Value" "GND"
-			(at 90.17 82.5499 90)
+			(at 123.19 74.9299 90)
 			(effects
 				(font
@@
 		)
 		(property "Footprint" ""
-			(at 93.98 82.55 0)
+			(at 127 74.93 0)
 			(effects
 				(font
@@
 		)
 		(property "Datasheet" ""
-			(at 93.98 82.55 0)
+			(at 127 74.93 0)
 			(effects
 				(font
@@
 		)
 		(property "Description" "Power symbol creates a global label with name \"GND\" , ground"
-			(at 93.98 82.55 0)
+			(at 127 74.93 0)
 			(effects
 				(font
@@
 	(symbol
 		(lib_id "custom library:BM04B-GHS-TBT")
-		(at 93.98 74.93 0)
+		(at 127 67.31 0)
 		(unit 1)
 		(exclude_from_sim no)
@@
 		(fields_autoplaced yes)
 		(property "Reference" "J3"
-			(at 107.95 77.4699 0)
+			(at 140.97 69.8499 0)
 			(effects
 				(font
@@
 		)
 		(property "Value" "BM04B-GHS-TBT"
-			(at 107.95 80.0099 0)
+			(at 140.97 72.3899 0)
 			(effects
 				(font
@@
 		)
 		(property "Footprint" "CONN_BM04B-GHS-TBT_JST"
-			(at 93.98 74.93 0)
+			(at 127 67.31 0)
 			(effects
 				(font
@@
 		)
 		(property "Datasheet" "BM04B-GHS-TBT"
-			(at 93.98 74.93 0)
+			(at 127 67.31 0)
 			(effects
 				(font
@@
 		)
 		(property "Description" ""
-			(at 93.98 74.93 0)
+			(at 127 67.31 0)
 			(effects
 				(font
@@
 	(symbol
 		(lib_id "power:+5V")
-		(at 93.98 74.93 90)
+		(at 127 67.31 90)
 		(unit 1)
 		(exclude_from_sim no)
@@
 		(fields_autoplaced yes)
 		(property "Reference" "#PWR015"
-			(at 97.79 74.93 0)
+			(at 130.81 67.31 0)
 			(effects
 				(font
@@
 		)
 		(property "Value" "+5V"
-			(at 90.17 74.9299 90)
+			(at 123.19 67.3099 90)
 			(effects
 				(font
@@
 		)
 		(property "Footprint" ""
-			(at 93.98 74.93 0)
+			(at 127 67.31 0)
 			(effects
 				(font
@@
 		)
 		(property "Datasheet" ""
-			(at 93.98 74.93 0)
+			(at 127 67.31 0)
 			(effects
 				(font
@@
 		)
 		(property "Description" "Power symbol creates a global label with name \"+5V\""
-			(at 93.98 74.93 0)
-			(effects
-				(font
+			(at 127 67.31 0)
+			(effects
+				(font

Commit message: started routing
Parts:
- J3: footprint CONN_BM04B-GHS-TBT_JST -> custom library:CONN_BM04B-GHS-TBT_JST
Connections:
- net +3.3V is gone; now on net +5V: J6.3 (Pin_3)
Changed lines of the file:
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@@
 	)
 	(symbol
-		(lib_id "power:+3.3V")
+		(lib_id "power:GND")
+		(at 127 74.93 270)
+		(unit 1)
+		(exclude_from_sim no)
+		(in_bom yes)
+		(on_board yes)
+		(dnp no)
+		(fields_autoplaced yes)
+		(property "Reference" "#PWR016"
+			(at 120.65 74.93 0)
+			(effects
+				(font
+					(size 1.27 1.27)
+				)
+				(hide yes)
+			)
+		)
+		(property "Value" "GND"
+			(at 123.19 74.9299 90)
+			(effects
+				(font
+					(size 1.27 1.27)
+				)
+				(justify right)
+			)
+		)
+		(property "Footprint" ""
+			(at 127 74.93 0)
+			(effects
+				(font
+					(size 1.27 1.27)
+				)
+				(hide yes)
+			)
+		)
+		(property "Datasheet" ""
+			(at 127 74.93 0)
+			(effects
+				(font
+					(size 1.27 1.27)
+				)
+				(hide yes)
+			)
+		)
+		(property "Description" "Power symbol creates a global label with name \"GND\" , ground"
+			(at 127 74.93 0)
+			(effects
+				(font
+					(size 1.27 1.27)
+				)
+				(hide yes)
+			)
+		)
+		(pin "1"
+		)
+		(instances
+			(project ""
+				(path "/b20a486a-db1b-4621-abfe-a5d205c676b3/52c764d6-917f-4b2b-b6f8-6c902b5ee893"
+					(reference "#PWR016")
+					(unit 1)
+				)
+			)
+		)
+	)
+	(symbol
+		(lib_id "power:+5V")
 		(at 121.92 52.07 90)
 		(unit 1)
@@
 			)
 		)
-		(property "Value" "+3.3V"
+		(property "Value" "+5V"
 			(at 118.11 52.0699 90)
 			(effects
@@
 			)
 		)
-		(property "Description" "Power symbol creates a global label with name \"+3.3V\""
+		(property "Description" "Power symbol creates a global label with name \"+5V\""
 			(at 121.92 52.07 0)
 			(effects
@@
 	(symbol
 		(lib_id "power:GND")
-		(at 127 74.93 270)
-		(unit 1)
-		(exclude_from_sim no)
-		(in_bom yes)
-		(on_board yes)
-		(dnp no)
-		(fields_autoplaced yes)
-		(property "Reference" "#PWR016"
-			(at 120.65 74.93 0)
-			(effects
-				(font
-					(size 1.27 1.27)
-				)
-				(hide yes)
-			)
-		)
-		(property "Value" "GND"
-			(at 123.19 74.9299 90)
-			(effects
-				(font
-					(size 1.27 1.27)
-				)
-				(justify right)
-			)
-		)
-		(property "Footprint" ""
-			(at 127 74.93 0)
-			(effects
-				(font
-					(size 1.27 1.27)
-				)
-				(hide yes)
-			)
-		)
-		(property "Datasheet" ""
-			(at 127 74.93 0)
-			(effects
-				(font
-					(size 1.27 1.27)
-				)
-				(hide yes)
-			)
-		)
-		(property "Description" "Power symbol creates a global label with name \"GND\" , ground"
-			(at 127 74.93 0)
-			(effects
-				(font
-					(size 1.27 1.27)
-				)
-				(hide yes)
-			)
-		)
-		(pin "1"
-		)
-		(instances
-			(project ""
-				(path "/b20a486a-db1b-4621-abfe-a5d205c676b3/52c764d6-917f-4b2b-b6f8-6c902b5ee893"
-					(reference "#PWR016")
-					(unit 1)
-				)
-			)
-		)
-	)
-	(symbol
-		(lib_id "power:GND")
 		(at 121.92 54.61 270)
 		(unit 1)
@@
 			)
 		)
-		(property "Footprint" "CONN_BM04B-GHS-TBT_JST"
+		(property "Footprint" "custom library:CONN_BM04B-GHS-TBT_JST"
 			(at 127 67.31 0)
 			(effects

Commit message: basically done
Parts:
- renumbered J3 to J1, J6 to J4
Changed lines of the file:
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@@
 		(dnp no)
 		(fields_autoplaced yes)
-		(property "Reference" "J6"
+		(property "Reference" "J4"
 			(at 128.27 49.5299 0)
 			(effects
@@
 			(project ""
 				(path "/b20a486a-db1b-4621-abfe-a5d205c676b3/52c764d6-917f-4b2b-b6f8-6c902b5ee893"
-					(reference "J6")
+					(reference "J4")
 					(unit 1)
 				)
@@
 		(dnp no)
 		(fields_autoplaced yes)
-		(property "Reference" "J3"
+		(property "Reference" "J1"
 			(at 140.97 69.8499 0)
 			(effects
@@
 			(project ""
 				(path "/b20a486a-db1b-4621-abfe-a5d205c676b3/52c764d6-917f-4b2b-b6f8-6c902b5ee893"
-					(reference "J3")
-					(unit 1)
-				)
+					(reference "J1")
+					(unit 1)
+				)
