File: MCU and Pi Board/mcu and pi board/servo power.kicad_sch (KiCad schematic)
At the start: 21 parts, among them IC3 CSD17578Q3A, IC4 CSD17578Q3A, U4 TPS40305DRCR

Commit message: started routing
Parts:
- C28, C29, C30, C31, C36: footprint (none) -> Capacitor_SMD:C_0805_2012Metric_Pad1.18x1.45mm_HandSolder
- C32, C33, C34, C37: footprint (none) -> Capacitor_SMD:C_0603_1608Metric_Pad1.08x0.95mm_HandSolder
- C35: value 100n -> 0.1u; footprint (none) -> Capacitor_SMD:C_0603_1608Metric_Pad1.08x0.95mm_HandSolder
- C38: footprint (none) -> Capacitor_SMD:C_1206_3216Metric_Pad1.33x1.80mm_HandSolder
- IC3, IC4: footprint CSD17578Q3A:TRANS_CSD18543Q3A -> custom library:TRANS_CSD18543Q3A
- R11, R12, R13, R14, R15, R16: footprint (none) -> Resistor_SMD:R_0603_1608Metric_Pad0.98x0.95mm_HandSolder
- U4: footprint DRC10_2P4X1P65 -> custom library:DRC10_2P4X1P65
Changed lines of the file:
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@@
 			)
 		)
-		(property "Footprint" ""
+		(property "Footprint" "Resistor_SMD:R_0603_1608Metric_Pad0.98x0.95mm_HandSolder"
 			(at 191.516 108.204 90)
 			(effects
@@
 			)
 		)
-		(property "Footprint" ""
+		(property "Footprint" "Capacitor_SMD:C_1206_3216Metric_Pad1.33x1.80mm_HandSolder"
 			(at 229.5652 93.98 0)
 			(effects
@@
 			)
 		)
-		(property "Footprint" ""
+		(property "Footprint" "Capacitor_SMD:C_0805_2012Metric_Pad1.18x1.45mm_HandSolder"
 			(at 74.6252 81.28 0)
 			(effects
@@
 			)
 		)
-		(property "Footprint" ""
+		(property "Footprint" "Capacitor_SMD:C_0603_1608Metric_Pad1.08x0.95mm_HandSolder"
 			(at 209.2452 104.14 0)
 			(effects
@@
 			)
 		)
-		(property "Footprint" ""
+		(property "Footprint" "Capacitor_SMD:C_0805_2012Metric_Pad1.18x1.45mm_HandSolder"
 			(at 58.1152 69.85 0)
 			(effects
@@
 			)
 		)
-		(property "Footprint" "CSD17578Q3A:TRANS_CSD18543Q3A"
+		(property "Footprint" "custom library:TRANS_CSD18543Q3A"
 			(at 209.55 63.5 0)
 			(effects
@@
 			)
 		)
-		(property "Footprint" "CSD17578Q3A:TRANS_CSD18543Q3A"
+		(property "Footprint" "custom library:TRANS_CSD18543Q3A"
 			(at 153.67 102.87 0)
 			(effects
@@
 			)
 		)
-		(property "Footprint" ""
+		(property "Footprint" "Resistor_SMD:R_0603_1608Metric_Pad0.98x0.95mm_HandSolder"
 			(at 209.296 92.964 90)
 			(effects
@@
 			)
 		)
-		(property "Footprint" ""
+		(property "Footprint" "Capacitor_SMD:C_0805_2012Metric_Pad1.18x1.45mm_HandSolder"
 			(at 191.4652 105.41 0)
 			(effects
@@
 			)
 		)
-		(property "Footprint" ""
+		(property "Footprint" "Resistor_SMD:R_0603_1608Metric_Pad0.98x0.95mm_HandSolder"
 			(at 123.444 99.314 90)
 			(effects
@@
 			)
 		)
-		(property "Footprint" ""
+		(property "Footprint" "Capacitor_SMD:C_0805_2012Metric_Pad1.18x1.45mm_HandSolder"
 			(at 72.0852 69.85 0)
 			(effects
@@
 			)
 		)
-		(property "Footprint" ""
+		(property "Footprint" "Capacitor_SMD:C_0805_2012Metric_Pad1.18x1.45mm_HandSolder"
 			(at 45.4152 69.85 0)
 			(effects
@@
 			)
 		)
-		(property "Footprint" ""
+		(property "Footprint" "Capacitor_SMD:C_0603_1608Metric_Pad1.08x0.95mm_HandSolder"
 			(at 180.0352 107.95 0)
 			(effects
@@
 			)
 		)
-		(property "Footprint" ""
+		(property "Footprint" "Capacitor_SMD:C_0603_1608Metric_Pad1.08x0.95mm_HandSolder"
 			(at 84.7852 69.85 0)
 			(effects
@@
 			)
 		)
-		(property "Footprint" ""
+		(property "Footprint" "Resistor_SMD:R_0603_1608Metric_Pad0.98x0.95mm_HandSolder"
 			(at 219.456 108.204 90)
 			(effects
@@
 			)
 		)
-		(property "Footprint" ""
+		(property "Footprint" "Resistor_SMD:R_0603_1608Metric_Pad0.98x0.95mm_HandSolder"
 			(at 219.456 92.964 90)
 			(effects
@@
 			)
 		)
-		(property "Value" "100n"
+		(property "Value" "0.1u"
 			(at 184.15 91.4399 0)
 			(effects
@@
 			)
 		)
-		(property "Footprint" ""
+		(property "Footprint" "Capacitor_SMD:C_0603_1608Metric_Pad1.08x0.95mm_HandSolder"
 			(at 181.3052 93.98 0)
 			(effects
@@
 			)
 		)
-		(property "Footprint" "DRC10_2P4X1P65"
+		(property "Footprint" "custom library:DRC10_2P4X1P65"
 			(at 96.52 66.04 0)
 			(effects
@@
 			)
 		)
-		(property "Footprint" ""
+		(property "Footprint" "Capacitor_SMD:C_0603_1608Metric_Pad1.08x0.95mm_HandSolder"
 			(at 88.5952 100.33 0)
 			(effects
@@
 			)
 		)
-		(property "Footprint" ""
+		(property "Footprint" "Resistor_SMD:R_0603_1608Metric_Pad0.98x0.95mm_HandSolder"
 			(at 88.646 84.074 90)
 			(effects

Commit message: basically done
Parts:
- renumbered C31 to C20, C35 to C23, C34 to C24, C36 to C25, C33 to C26, C37 to C27, C29 to C31, C32 to C33, IC4 to IC1, IC3 to IC2, L2 to L1, R13 to R10, R15 to R12, R12 to R13, R16 to R9, U4 to U7
Changed lines of the file:
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@@
 		(dnp no)
 		(fields_autoplaced yes)
-		(property "Reference" "R13"
+		(property "Reference" "R10"
 			(at 193.04 106.6799 0)
 			(effects
@@
 			(project "mcu and pi board"
 				(path "/b20a486a-db1b-4621-abfe-a5d205c676b3/bef0208e-671a-46f7-958e-767cd5c13c2b/4dcaefb5-a695-4167-8329-a8d078427477"
-					(reference "R13")
+					(reference "R10")
 					(unit 1)
 				)
@@
 		(dnp no)
 		(fields_autoplaced yes)
-		(property "Reference" "L2"
+		(property "Reference" "L1"
 			(at 186.69 76.2 90)
 			(effects
@@
 			(project "mcu and pi board"
 				(path "/b20a486a-db1b-4621-abfe-a5d205c676b3/bef0208e-671a-46f7-958e-767cd5c13c2b/4dcaefb5-a695-4167-8329-a8d078427477"
-					(reference "L2")
+					(reference "L1")
 					(unit 1)
 				)
@@
 		(on_board yes)
 		(dnp no)
-		(property "Reference" "C31"
+		(property "Reference" "C20"
 			(at 77.47 76.1999 0)
 			(effects
@@
 			(project "mcu and pi board"
 				(path "/b20a486a-db1b-4621-abfe-a5d205c676b3/bef0208e-671a-46f7-958e-767cd5c13c2b/4dcaefb5-a695-4167-8329-a8d078427477"
-					(reference "C31")
+					(reference "C20")
 					(unit 1)
 				)
@@
 		(on_board yes)
 		(dnp no)
-		(property "Reference" "C37"
+		(property "Reference" "C27"
 			(at 212.09 99.0599 0)
 			(effects
@@
 			(project "mcu and pi board"
 				(path "/b20a486a-db1b-4621-abfe-a5d205c676b3/bef0208e-671a-46f7-958e-767cd5c13c2b/4dcaefb5-a695-4167-8329-a8d078427477"
-					(reference "C37")
+					(reference "C27")
 					(unit 1)
 				)
@@
 		(on_board yes)
 		(dnp no)
-		(property "Reference" "C29"
+		(property "Reference" "C31"
 			(at 60.96 64.7699 0)
 			(effects
@@
 			(project "mcu and pi board"
 				(path "/b20a486a-db1b-4621-abfe-a5d205c676b3/bef0208e-671a-46f7-958e-767cd5c13c2b/4dcaefb5-a695-4167-8329-a8d078427477"
-					(reference "C29")
+					(reference "C31")
 					(unit 1)
 				)
@@
 		(dnp no)
 		(fields_autoplaced yes)
-		(property "Reference" "IC4"
+		(property "Reference" "IC1"
 			(at 209.55 45.72 0)
 			(effects
@@
 			(project "mcu and pi board"
 				(path "/b20a486a-db1b-4621-abfe-a5d205c676b3/bef0208e-671a-46f7-958e-767cd5c13c2b/4dcaefb5-a695-4167-8329-a8d078427477"
-					(reference "IC4")
+					(reference "IC1")
 					(unit 1)
 				)
@@
 		(dnp no)
 		(fields_autoplaced yes)
-		(property "Reference" "IC3"
+		(property "Reference" "IC2"
 			(at 153.67 85.09 0)
 			(effects
@@
 			(project "mcu and pi board"
 				(path "/b20a486a-db1b-4621-abfe-a5d205c676b3/bef0208e-671a-46f7-958e-767cd5c13c2b/4dcaefb5-a695-4167-8329-a8d078427477"
-					(reference "IC3")
+					(reference "IC2")
 					(unit 1)
 				)
@@
 		(on_board yes)
 		(dnp no)
-		(property "Reference" "C36"
+		(property "Reference" "C25"
 			(at 194.31 100.3299 0)
 			(effects
@@
 			(project "mcu and pi board"
 				(path "/b20a486a-db1b-4621-abfe-a5d205c676b3/bef0208e-671a-46f7-958e-767cd5c13c2b/4dcaefb5-a695-4167-8329-a8d078427477"
-					(reference "C36")
+					(reference "C25")
 					(unit 1)
 				)
@@
 		(dnp no)
 		(fields_autoplaced yes)
-		(property "Reference" "R12"
+		(property "Reference" "R13"
 			(at 123.19 93.98 90)
 			(effects
@@
 			(project "mcu and pi board"
 				(path "/b20a486a-db1b-4621-abfe-a5d205c676b3/bef0208e-671a-46f7-958e-767cd5c13c2b/4dcaefb5-a695-4167-8329-a8d078427477"
-					(reference "R12")
+					(reference "R13")
 					(unit 1)
 				)
@@
 		(on_board yes)
 		(dnp no)
-		(property "Reference" "C34"
+		(property "Reference" "C24"
 			(at 182.88 102.8699 0)
 			(effects
@@
 			(project "mcu and pi board"
 				(path "/b20a486a-db1b-4621-abfe-a5d205c676b3/bef0208e-671a-46f7-958e-767cd5c13c2b/4dcaefb5-a695-4167-8329-a8d078427477"
-					(reference "C34")
+					(reference "C24")
 					(unit 1)
 				)
@@
 		(on_board yes)
 		(dnp no)
-		(property "Reference" "C32"
+		(property "Reference" "C33"
 			(at 87.63 64.7699 0)
 			(effects
@@
 			(project "mcu and pi board"
 				(path "/b20a486a-db1b-4621-abfe-a5d205c676b3/bef0208e-671a-46f7-958e-767cd5c13c2b/4dcaefb5-a695-4167-8329-a8d078427477"
-					(reference "C32")
+					(reference "C33")
 					(unit 1)
 				)
@@
 		(dnp no)
 		(fields_autoplaced yes)
-		(property "Reference" "R16"
+		(property "Reference" "R9"
 			(at 220.98 106.6799 0)
 			(effects
@@
 			(project "mcu and pi board"
 				(path "/b20a486a-db1b-4621-abfe-a5d205c676b3/bef0208e-671a-46f7-958e-767cd5c13c2b/4dcaefb5-a695-4167-8329-a8d078427477"
-					(reference "R16")
+					(reference "R9")
 					(unit 1)
 				)
@@
 		(dnp no)
 		(fields_autoplaced yes)
-		(property "Reference" "R15"
+		(property "Reference" "R12"
 			(at 220.98 91.4399 0)
 			(effects
@@
 			(project "mcu and pi board"
 				(path "/b20a486a-db1b-4621-abfe-a5d205c676b3/bef0208e-671a-46f7-958e-767cd5c13c2b/4dcaefb5-a695-4167-8329-a8d078427477"
-					(reference "R15")
+					(reference "R12")
 					(unit 1)
 				)
@@
 		(on_board yes)
 		(dnp no)
-		(property "Reference" "C35"
+		(property "Reference" "C23"
 			(at 184.15 88.8999 0)
 			(effects
@@
 			(project "mcu and pi board"
 				(path "/b20a486a-db1b-4621-abfe-a5d205c676b3/bef0208e-671a-46f7-958e-767cd5c13c2b/4dcaefb5-a695-4167-8329-a8d078427477"
-					(reference "C35")
+					(reference "C23")
 					(unit 1)
 				)
@@
 		(dnp no)
 		(fields_autoplaced yes)
-		(property "Reference" "U4"
+		(property "Reference" "U7"
 			(at 132.08 55.88 0)
 			(effects
@@
 			(project "mcu and pi board"
 				(path "/b20a486a-db1b-4621-abfe-a5d205c676b3/bef0208e-671a-46f7-958e-767cd5c13c2b/4dcaefb5-a695-4167-8329-a8d078427477"
-					(reference "U4")
+					(reference "U7")
 					(unit 1)
 				)
@@
 		(on_board yes)
 		(dnp no)
-		(property "Reference" "C33"
+		(property "Reference" "C26"
 			(at 91.44 95.2499 0)
 			(effects
@@
 			(project "mcu and pi board"
 				(path "/b20a486a-db1b-4621-abfe-a5d205c676b3/bef0208e-671a-46f7-958e-767cd5c13c2b/4dcaefb5-a695-4167-8329-a8d078427477"
-					(reference "C33")
-					(unit 1)
-				)
+					(reference "C26")
+					(unit 1)
+				)
