File: MCU and Pi Board/mcu and pi board/stm32.kicad_sch (KiCad schematic)
At the start: 28 parts, among them J15 Conn_01x28_Socket, J16 Conn_01x28_Socket, J17 DebugnBoot, J18 UART-PINS, J19 Conn_01x02_Pin, J20 Conn_01x03_Pin, J21 Conn_01x05, J26 Conn_01x03_Pin, J27 Conn_01x02_Pin, J30 Conn_01x04_Pin, J31 Conn_01x04_Pin, J32 Conn_01x02_Pin, J33 Conn_01x02_Pin, J34 Conn_01x03_Pin, J7 Conn_01x04_Pin, U1 STM32F091CCT6

Commit message: basically done
Parts:
- U3: renamed from U1; footprint LQFP48-7x7mm -> custom library:LQFP48-7x7mm
- renumbered C13 to C14, C11 to C15, C14 to C16, C15 to C17, C12 to C18, C16 to C19, J31 to J11, J19 to J12, J34 to J13, J16 to J15, J15 to J16, J27 to J17, J7 to J18, J20 to J19, J30 to J20, J33 to J21, J17 to J27, J18 to J28, J32 to J8, J21 to J9, R3 to R4, R18 to R5, R19 to R6, R1 to R7, R2 to R8
Changed lines of the file:
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@@
 		(dnp no)
 		(fields_autoplaced yes)
-		(property "Reference" "R3"
+		(property "Reference" "R4"
 			(at 62.23 64.7699 0)
 			(effects
@@
 			(project ""
 				(path "/b20a486a-db1b-4621-abfe-a5d205c676b3/51029924-342a-47f7-95d8-8f14ebe6a876"
-					(reference "R3")
+					(reference "R4")
 					(unit 1)
 				)
@@
 		(dnp no)
 		(fields_autoplaced yes)
-		(property "Reference" "J20"
+		(property "Reference" "J19"
 			(at 227.965 87.63 0)
 			(effects
@@
 			(project ""
 				(path "/b20a486a-db1b-4621-abfe-a5d205c676b3/51029924-342a-47f7-95d8-8f14ebe6a876"
-					(reference "J20")
+					(reference "J19")
 					(unit 1)
 				)
@@
 		(on_board yes)
 		(dnp no)
-		(property "Reference" "J16"
+		(property "Reference" "J15"
 			(at 27.94 101.346 0)
 			(effects
@@
 			(project "mcu and pi board"
 				(path "/b20a486a-db1b-4621-abfe-a5d205c676b3/51029924-342a-47f7-95d8-8f14ebe6a876"
-					(reference "J16")
+					(reference "J15")
 					(unit 1)
 				)
@@
 		(on_board yes)
 		(dnp no)
-		(property "Reference" "C13"
+		(property "Reference" "C14"
 			(at 243.84 47.244 90)
 			(effects
@@
 			(project "mcu and pi board"
 				(path "/b20a486a-db1b-4621-abfe-a5d205c676b3/51029924-342a-47f7-95d8-8f14ebe6a876"
-					(reference "C13")
+					(reference "C14")
 					(unit 1)
 				)
@@
 		(dnp no)
 		(fields_autoplaced yes)
-		(property "Reference" "J17"
+		(property "Reference" "J27"
 			(at 138.43 163.8299 0)
 			(effects
@@
 			(project "mcu and pi board"
 				(path "/b20a486a-db1b-4621-abfe-a5d205c676b3/51029924-342a-47f7-95d8-8f14ebe6a876"
-					(reference "J17")
+					(reference "J27")
 					(unit 1)
 				)
@@
 		(on_board yes)
 		(dnp no)
-		(property "Reference" "J18"
+		(property "Reference" "J28"
 			(at 141.224 176.53 0)
 			(effects
@@
 			(project "mcu and pi board"
 				(path "/b20a486a-db1b-4621-abfe-a5d205c676b3/51029924-342a-47f7-95d8-8f14ebe6a876"
-					(reference "J18")
+					(reference "J28")
 					(unit 1)
 				)
@@
 		(on_board yes)
 		(dnp no)
-		(property "Reference" "C15"
+		(property "Reference" "C17"
 			(at 244.094 61.468 90)
 			(effects
@@
 			(project "mcu and pi board"
 				(path "/b20a486a-db1b-4621-abfe-a5d205c676b3/51029924-342a-47f7-95d8-8f14ebe6a876"
-					(reference "C15")
+					(reference "C17")
 					(unit 1)
 				)
@@
 		(dnp no)
 		(fields_autoplaced yes)
-		(property "Reference" "J30"
+		(property "Reference" "J20"
 			(at 168.275 107.95 0)
 			(effects
@@
 			(project ""
 				(path "/b20a486a-db1b-4621-abfe-a5d205c676b3/51029924-342a-47f7-95d8-8f14ebe6a876"
-					(reference "J30")
+					(reference "J20")
 					(unit 1)
 				)
@@
 		(dnp no)
 		(fields_autoplaced yes)
-		(property "Reference" "R19"
+		(property "Reference" "R6"
 			(at 73.66 21.5899 0)
 			(effects
@@
 			(project "mcu and pi board"
 				(path "/b20a486a-db1b-4621-abfe-a5d205c676b3/51029924-342a-47f7-95d8-8f14ebe6a876"
-					(reference "R19")
+					(reference "R6")
 					(unit 1)
 				)
@@
 		(dnp no)
 		(fields_autoplaced yes)
-		(property "Reference" "C11"
+		(property "Reference" "C15"
 			(at 96.52 49.5299 0)
 			(effects
@@
 			(project ""
 				(path "/b20a486a-db1b-4621-abfe-a5d205c676b3/51029924-342a-47f7-95d8-8f14ebe6a876"
-					(reference "C11")
+					(reference "C15")
 					(unit 1)
 				)
@@
 		(dnp no)
 		(fields_autoplaced yes)
-		(property "Reference" "U1"
+		(property "Reference" "U3"
 			(at 128.27 41.91 0)
 			(effects
@@
 			)
 		)
-		(property "Footprint" "LQFP48-7x7mm"
+		(property "Footprint" "custom library:LQFP48-7x7mm"
 			(at 102.87 54.61 0)
 			(effects
@@
 			(project ""
 				(path "/b20a486a-db1b-4621-abfe-a5d205c676b3/51029924-342a-47f7-95d8-8f14ebe6a876"
-					(reference "U1")
+					(reference "U3")
 					(unit 1)
 				)
@@
 		(dnp no)
 		(fields_autoplaced yes)
-		(property "Reference" "J32"
+		(property "Reference" "J8"
 			(at 234.315 113.03 0)
 			(effects
@@
 			(project "mcu and pi board"
 				(path "/b20a486a-db1b-4621-abfe-a5d205c676b3/51029924-342a-47f7-95d8-8f14ebe6a876"
-					(reference "J32")
+					(reference "J8")
 					(unit 1)
 				)
@@
 		(dnp no)
 		(fields_autoplaced yes)
-		(property "Reference" "J21"
+		(property "Reference" "J9"
 			(at 176.53 156.2099 0)
 			(effects
@@
 			(project ""
 				(path "/b20a486a-db1b-4621-abfe-a5d205c676b3/51029924-342a-47f7-95d8-8f14ebe6a876"
-					(reference "J21")
+					(reference "J9")
 					(unit 1)
 				)
@@
 		(dnp no)
 		(fields_autoplaced yes)
-		(property "Reference" "R1"
+		(property "Reference" "R7"
 			(at 67.31 48.26 90)
 			(effects
@@
 			(project ""
 				(path "/b20a486a-db1b-4621-abfe-a5d205c676b3/51029924-342a-47f7-95d8-8f14ebe6a876"
-					(reference "R1")
+					(reference "R7")
 					(unit 1)
 				)
@@
 		(on_board yes)
 		(dnp no)
-		(property "Reference" "C16"
+		(property "Reference" "C19"
 			(at 244.094 56.388 90)
 			(effects
@@
 			(project "mcu and pi board"
 				(path "/b20a486a-db1b-4621-abfe-a5d205c676b3/51029924-342a-47f7-95d8-8f14ebe6a876"
-					(reference "C16")
+					(reference "C19")
 					(unit 1)
 				)
@@
 		(dnp no)
 		(fields_autoplaced yes)
-		(property "Reference" "J19"
+		(property "Reference" "J12"
 			(at 206.375 105.41 0)
 			(effects
@@
 			(project ""
 				(path "/b20a486a-db1b-4621-abfe-a5d205c676b3/51029924-342a-47f7-95d8-8f14ebe6a876"
-					(reference "J19")
+					(reference "J12")
 					(unit 1)
 				)
@@
 		(dnp no)
 		(fields_autoplaced yes)
-		(property "Reference" "R2"
+		(property "Reference" "R8"
 			(at 88.9 96.52 90)
 			(effects
@@
 			(project ""
 				(path "/b20a486a-db1b-4621-abfe-a5d205c676b3/51029924-342a-47f7-95d8-8f14ebe6a876"
-					(reference "R2")
+					(reference "R8")
 					(unit 1)
 				)
@@
 		(dnp no)
 		(fields_autoplaced yes)
-		(property "Reference" "U1"
+		(property "Reference" "U3"
 			(at 181.61 52.0701 0)
 			(effects
@@
 			)
 		)
-		(property "Footprint" "LQFP48-7x7mm"
+		(property "Footprint" "custom library:LQFP48-7x7mm"
 			(at 215.9 62.23 0)
 			(effects
@@
 			(project ""
 				(path "/b20a486a-db1b-4621-abfe-a5d205c676b3/51029924-342a-47f7-95d8-8f14ebe6a876"
-					(reference "U1")
+					(reference "U3")
 					(unit 2)
 				)
@@
 		(dnp no)
 		(fields_autoplaced yes)
-		(property "Reference" "C12"
+		(property "Reference" "C18"
 			(at 236.22 35.56 90)
 			(effects
@@
 			(project ""
 				(path "/b20a486a-db1b-4621-abfe-a5d205c676b3/51029924-342a-47f7-95d8-8f14ebe6a876"
-					(reference "C12")
+					(reference "C18")
 					(unit 1)
 				)
@@
 		(dnp no)
 		(fields_autoplaced yes)
-		(property "Reference" "J34"
+		(property "Reference" "J13"
 			(at 178.435 93.98 0)
 			(effects
@@
 			(project "mcu and pi board"
 				(path "/b20a486a-db1b-4621-abfe-a5d205c676b3/51029924-342a-47f7-95d8-8f14ebe6a876"
-					(reference "J34")
+					(reference "J13")
 					(unit 1)
 				)
@@
 		(dnp no)
 		(fields_autoplaced yes)
-		(property "Reference" "J7"
+		(property "Reference" "J18"
 			(at 121.285 115.57 0)
 			(effects
@@
 			(project ""
 				(path "/b20a486a-db1b-4621-abfe-a5d205c676b3/51029924-342a-47f7-95d8-8f14ebe6a876"
-					(reference "J7")
+					(reference "J18")
 					(unit 1)
 				)
@@
 		(dnp no)
 		(fields_autoplaced yes)
-		(property "Reference" "R18"
+		(property "Reference" "R5"
 			(at 111.76 147.32 90)
 			(effects
@@
 			(project "mcu and pi board"
 				(path "/b20a486a-db1b-4621-abfe-a5d205c676b3/51029924-342a-47f7-95d8-8f14ebe6a876"
-					(reference "R18")
+					(reference "R5")
 					(unit 1)
 				)
@@
 		(dnp no)
 		(fields_autoplaced yes)
-		(property "Reference" "J31"
+		(property "Reference" "J11"
 			(at 191.135 121.92 0)
 			(effects
@@
 			(project "mcu and pi board"
 				(path "/b20a486a-db1b-4621-abfe-a5d205c676b3/51029924-342a-47f7-95d8-8f14ebe6a876"
-					(reference "J31")
+					(reference "J11")
 					(unit 1)
 				)
@@
 		(dnp no)
 		(fields_autoplaced yes)
-		(property "Reference" "J27"
+		(property "Reference" "J17"
 			(at 220.345 123.19 0)
 			(effects
@@
 			(project ""
 				(path "/b20a486a-db1b-4621-abfe-a5d205c676b3/51029924-342a-47f7-95d8-8f14ebe6a876"
-					(reference "J27")
+					(reference "J17")
 					(unit 1)
 				)
@@
 		(on_board yes)
 		(dnp no)
-		(property "Reference" "C14"
+		(property "Reference" "C16"
 			(at 244.094 66.548 90)
 			(effects
@@
 			(project "mcu and pi board"
 				(path "/b20a486a-db1b-4621-abfe-a5d205c676b3/51029924-342a-47f7-95d8-8f14ebe6a876"
-					(reference "C14")
+					(reference "C16")
 					(unit 1)
 				)
@@
 		(dnp no)
 		(fields_autoplaced yes)
-		(property "Reference" "J33"
+		(property "Reference" "J21"
 			(at 225.425 74.93 0)
 			(effects
@@
 			(project ""
 				(path "/b20a486a-db1b-4621-abfe-a5d205c676b3/51029924-342a-47f7-95d8-8f14ebe6a876"
-					(reference "J33")
+					(reference "J21")
 					(unit 1)
 				)
@@
 		(on_board yes)
 		(dnp no)
-		(property "Reference" "J15"
+		(property "Reference" "J16"
 			(at 49.276 101.854 0)
 			(effects
@@
 			(project ""
 				(path "/b20a486a-db1b-4621-abfe-a5d205c676b3/51029924-342a-47f7-95d8-8f14ebe6a876"
-					(reference "J15")
+					(reference "J16")
 					(unit 1)
 				)
