File: MCU and Pi Board/mcu and pi board/stm32.kicad_sch (KiCad schematic)
At the start: 28 parts, among them J11 Conn_01x04_Pin, J12 Conn_01x02_Pin, J13 Conn_01x03_Pin, J15 Conn_01x28_Socket, J16 Conn_01x28_Socket, J17 Conn_01x02_Pin, J18 Conn_01x04_Pin, J19 Conn_01x03_Pin, J20 Conn_01x04_Pin, J21 Conn_01x02_Pin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

Commit message: bom updated stuff
Parts:
- C14, C15, C16, C17, C18, C19: Voltage Rating (none) -> 10V
Changed lines of the file:
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@@
+			)
+		)
+		(property "Voltage Rating" "10V"
+			(at 236.22 49.53 90)
+			(effects
+				(font
+					(size 1.27 1.27)
+				)
+				(hide yes)
 			)
 		)
@@
 			)
 		)
+		(property "Voltage Rating" "10V"
+			(at 236.22 62.23 90)
+			(effects
+				(font
+					(size 1.27 1.27)
+				)
+				(hide yes)
+			)
+		)
 		(pin "1"
 		)
@@
 			)
 		)
+		(property "Voltage Rating" "10V"
+			(at 92.71 50.8 0)
+			(effects
+				(font
+					(size 1.27 1.27)
+				)
+				(hide yes)
+			)
+		)
 		(pin "2"
 		)
@@
 			)
 		)
+		(property "Voltage Rating" "10V"
+			(at 236.22 57.15 90)
+			(effects
+				(font
+					(size 1.27 1.27)
+				)
+				(hide yes)
+			)
+		)
 		(pin "1"
 		)
@@
 			)
 		)
+		(property "Voltage Rating" "10V"
+			(at 236.22 43.18 90)
+			(effects
+				(font
+					(size 1.27 1.27)
+				)
+				(hide yes)
+			)
+		)
 		(pin "1"
 		)
@@
 			(effects
 				(font
+					(size 1.27 1.27)
+				)
+				(hide yes)
+			)
+		)
+		(property "Voltage Rating" "10V"
+			(at 236.22 67.31 90)
+			(effects
+				(font
