File: MCU and Pi Board/mcu and pi board/_autosave-power.kicad_sch (KiCad schematic)
At the start: 36 parts, among them J14 ET60T-D04-0-00-D04-X-R1-S, J2 ET60S-D04-3-08-D04-X-R1-S, J24 IPBT-105-H1-T-D-GP, J3 PJ-002A, J5 PJ-002A, J6 IPBT-105-H1-T-D-GP, Q1 BSC010N04LS6ATMA1, Q2 BSC010N04LS6ATMA1, U1 LTC4370CMS_PBF, U2 LM3940IMPX-3.3/NOPB

Commit message: bom updated stuff
Parts:
- R2: value 270 -> 100
Changed lines of the file:
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@@
 			)
 		)
-		(property "Value" "270"
+		(property "Value" "100"
 			(at 80.01 87.6299 0)
 			(effects
