File: MCU and Pi Board/mcu and pi board/pi.kicad_sch (KiCad schematic)
At the start: 6 parts, among them J12 430450428, J28 Conn_02x04_Counter_Clockwise, J35 Conn_02x09_Counter_Clockwise, U5 RASPBERRY_PI_4B_4GB

Commit message: basically done
Parts:
- renumbered C19 to C12, C18 to C13, J12 to J10, J35 to J25, J28 to J7, U5 to U4
Changed lines of the file:
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@@
 		(dnp no)
 		(fields_autoplaced yes)
-		(property "Reference" "J28"
+		(property "Reference" "J7"
 			(at 135.89 100.33 0)
 			(effects
@@
 			(project ""
 				(path "/b20a486a-db1b-4621-abfe-a5d205c676b3/dda479c6-78f4-4e1c-82b6-b799f08d03a6"
-					(reference "J28")
+					(reference "J7")
 					(unit 1)
 				)
@@
 		(dnp no)
 		(fields_autoplaced yes)
-		(property "Reference" "C18"
+		(property "Reference" "C13"
 			(at 248.92 41.9099 0)
 			(effects
@@
 			(project ""
 				(path "/b20a486a-db1b-4621-abfe-a5d205c676b3/dda479c6-78f4-4e1c-82b6-b799f08d03a6"
-					(reference "C18")
+					(reference "C13")
 					(unit 1)
 				)
@@
 		(dnp no)
 		(fields_autoplaced yes)
-		(property "Reference" "J35"
+		(property "Reference" "J25"
 			(at 104.14 67.31 0)
 			(effects
@@
 			(project ""
 				(path "/b20a486a-db1b-4621-abfe-a5d205c676b3/dda479c6-78f4-4e1c-82b6-b799f08d03a6"
-					(reference "J35")
+					(reference "J25")
 					(unit 1)
 				)
@@
 		(dnp no)
 		(fields_autoplaced yes)
-		(property "Reference" "J12"
+		(property "Reference" "J10"
 			(at 256.54 59.69 0)
 			(effects
@@
 			(project ""
 				(path "/b20a486a-db1b-4621-abfe-a5d205c676b3/dda479c6-78f4-4e1c-82b6-b799f08d03a6"
-					(reference "J12")
+					(reference "J10")
 					(unit 1)
 				)
@@
 		(dnp no)
 		(fields_autoplaced yes)
-		(property "Reference" "C19"
+		(property "Reference" "C12"
 			(at 233.68 41.9099 0)
 			(effects
@@
 			(project "mcu and pi board"
 				(path "/b20a486a-db1b-4621-abfe-a5d205c676b3/dda479c6-78f4-4e1c-82b6-b799f08d03a6"
-					(reference "C19")
+					(reference "C12")
 					(unit 1)
 				)
@@
 		(dnp no)
 		(fields_autoplaced yes)
-		(property "Reference" "U5"
+		(property "Reference" "U4"
 			(at 194.31 38.1 0)
 			(effects
@@
 			(project ""
 				(path "/b20a486a-db1b-4621-abfe-a5d205c676b3/dda479c6-78f4-4e1c-82b6-b799f08d03a6"
-					(reference "U5")
+					(reference "U4")
 					(unit 1)
 				)

Commit message: bom updated stuff
Parts:
- C12, C13: Voltage Rating (none) -> 10V
Changed lines of the file:
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@@
+			)
+		)
+		(property "Voltage Rating" "10V"
+			(at 245.11 43.18 0)
+			(effects
+				(font
+					(size 1.27 1.27)
+				)
+				(hide yes)
 			)
 		)
@@
 			(at 229.87 43.18 0)
 			(effects
+				(font
+					(size 1.27 1.27)
+				)
+				(hide yes)
+			)
+		)
+		(property "Voltage Rating" "10V"
+			(at 229.87 43.18 0)
+			(effects
