File: MCU and Pi Board/mcu and pi board/power.kicad_sch (KiCad schematic)
At the start: 36 parts, among them J14 ET60T-D04-0-00-D04-X-R1-S, J2 ET60S-D04-3-08-D04-X-R1-S, J24 IPBT-105-H1-T-D-GP, J3 PJ-002A, J5 PJ-002A, J6 IPBT-105-H1-T-D-GP, Q1 BSC010N04LS6ATMA1, Q2 BSC010N04LS6ATMA1, U1 LTC4370CMS_PBF, U2 LM3940IMPX-3.3/NOPB

Commit message: commit ig
Parts:
- R1: value 290 -> 330
- R16: value 200 -> 470
- R2: value 270 -> 100
- R3: value 510 -> 1k
Changed lines of the file:
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@@
 			)
 		)
-		(property "Value" "510"
+		(property "Value" "1k"
 			(at 86.36 149.8599 0)
 			(effects
@@
 			)
 		)
-		(property "Value" "270"
+		(property "Value" "100"
 			(at 80.01 87.6299 0)
 			(effects
@@
 			)
 		)
-		(property "Value" "290"
+		(property "Value" "330"
 			(at 96.52 126.9999 0)
 			(effects
@@
 			)
 		)
-		(property "Value" "200"
+		(property "Value" "470"
 			(at 64.77 99.0599 0)
 			(effects
